File: keeby.kicad_sch (KiCad schematic)
At the start: 0 parts

Commit message: Update
Other:
- added sheet left (half.kicad_sch)
- added sheet right (half.kicad_sch)
Changed lines of the file:
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@@
 	(generator_version "9.0")
 	(paper "A4")
+	(sheet
+		(at 154.94 61.722)
+		(size 90.424 48.26)
+		(exclude_from_sim no)
+		(in_bom yes)
+		(on_board yes)
+		(dnp no)
+		(fields_autoplaced yes)
+		(stroke
+			(width 0.1524)
+			(type solid)
+		)
+		(fill
+			(color 0 0 0 0.0000)
+		)
+		(property "Sheetname" "right"
+			(at 154.94 61.0104 0)
+			(effects
+				(font
+					(size 1.27 1.27)
+				)
+				(justify left bottom)
+			)
+		)
+		(property "Sheetfile" "half.kicad_sch"
+			(at 154.94 110.5666 0)
+			(effects
+				(font
+					(size 1.27 1.27)
+				)
+				(justify left top)
+			)
+		)
+		(instances
+			(project "keeby"
+				(path "/fade6638-4e22-4fdd-8807-944beeb130ad"
+					(page "3")
+				)
+			)
+		)
+	)
+	(sheet
+		(at 36.576 61.468)
+		(size 90.17 49.53)
+		(exclude_from_sim no)
+		(in_bom yes)
+		(on_board yes)
+		(dnp no)
+		(fields_autoplaced yes)
+		(stroke
+			(width 0.1524)
+			(type solid)
+		)
+		(fill
+			(color 0 0 0 0.0000)
+		)
+		(property "Sheetname" "left"
+			(at 36.576 60.7564 0)
+			(effects
+				(font
+					(size 1.27 1.27)
+				)
+				(justify left bottom)
+			)
+		)
+		(property "Sheetfile" "half.kicad_sch"
+			(at 36.576 111.5826 0)
+			(effects
+				(font
+					(size 1.27 1.27)
+				)
+				(justify left top)
+			)
+		)
+		(instances
+			(project "keeby"
+				(path "/fade6638-4e22-4fdd-8807-944beeb130ad"
+					(page "2")
+				)
+			)
+		)
+	)
 	(sheet_instances
 		(path "/"

Commit message: Update
Changed lines of the file:
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@@
 	(paper "A4")
 	(sheet
-		(at 154.94 61.722)
+		(at 158.75 38.1)
 		(size 90.424 48.26)
 		(exclude_from_sim no)
@@
 		)
 		(property "Sheetname" "right"
-			(at 154.94 61.0104 0)
+			(at 158.75 37.3884 0)
 			(effects
 				(font
@@
 		)
 		(property "Sheetfile" "half.kicad_sch"
-			(at 154.94 110.5666 0)
+			(at 158.75 86.9446 0)
 			(effects
 				(font
@@
 	)
 	(sheet
-		(at 36.576 61.468)
+		(at 40.64 38.1)
 		(size 90.17 49.53)
 		(exclude_from_sim no)
@@
 		)
 		(property "Sheetname" "left"
-			(at 36.576 60.7564 0)
+			(at 40.64 37.3884 0)
 			(effects
 				(font
@@
 		)
 		(property "Sheetfile" "half.kicad_sch"
-			(at 36.576 111.5826 0)
+			(at 40.64 88.2146 0)
 			(effects
 				(font
