File: half.kicad_sch (KiCad schematic)
At the start: 88 parts, among them J3 JST_PH, Q1 Q_PMOS_GSD, SW1 SW_Push, SW13 SW_Push, SW14 SW_Push, SW15 SW_Push, SW16 SW_Push, SW17 SW_Push, SW18 SW_Push, SW25 SW_Push, SW26 SW_Push, SW27 SW_Push, SW28 SW_Push, SW29 SW_Push, SW3 SW_Push, SW30 SW_Push, SW37 SW_Push, SW38 SW_Push, SW39 SW_Push, SW40 SW_Push, SW41 SW_Push, SW42 SW_Push, SW49 SW_Push, SW5 SW_Push, SW50 SW_Push, SW51 SW_Push, SW52 SW_Push, SW53 SW_Push, SW54 RotaryEncoder_Switch, SW61 SW_SPDT, SW7 SW_Push, SW8 SW_Push, SW9 SW_Push, U3 SuperMini nRF52840

Commit message: update
Parts:
- added D100, D103, D104, D107, D108, D111, D112, D115, D116, D99: SK6812MINI, LED_SMD:LED_SK6812MINI_PLCC4_3.5x3.5mm_P1.75mm, symbol LED:SK6812MINI
- added Q3: Q_NMOS_GSD, symbol Transistor_FET:Q_NMOS_GSD
- added R1: 1kΩ, Resistor_SMD:R_0805_2012Metric, symbol Device:R
Connections:
- net GND: now also D100.2 (VSS), D103.2 (VSS), D104.2 (VSS), D107.2 (VSS), D108.2 (VSS), D111.2 (VSS), D112.2 (VSS), D115.2 (VSS), D116.2 (VSS), D99.2 (VSS), Q3.2 (S)
- net LED_PWR: now also R1.1; no longer Q1.1 (G), R5.2
- net at D54.4 (VDD), D61.4 (VDD), D63.4 (VDD)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: now also D100.4 (VDD), D103.4 (VDD), D104.4 (VDD), D107.4 (VDD), D108.4 (VDD), D111.4 (VDD), D112.4 (VDD), D115.4 (VDD), D116.4 (VDD), D99.4 (VDD)
- net at D77.1 (DOUT): now also D99.3 (DIN); no longer D97.3 (DIN)
- new net: D100.3 (DIN), D104.1 (DOUT)
- new net: D104.3 (DIN), D108.1 (DOUT)
- new net: Q3.1 (G), R1.2
- new net: Q1.1 (G), Q3.3 (D), R5.2
- new net: D103.3 (DIN), D99.1 (DOUT)
- new net: D112.3 (DIN), D116.1 (DOUT)
- new net: D115.1 (DOUT), D116.3 (DIN)
- new net: D107.1 (DOUT), D111.3 (DIN)
- new net: D103.1 (DOUT), D107.3 (DIN)
- new net: D111.1 (DOUT), D115.3 (DIN)
- new net: D108.3 (DIN), D112.1 (DOUT)
- new net: D100.1 (DOUT), D97.3 (DIN)
- no-connect marks 0 -> 1
Other:
- moved on the sheet: D54, D61, D63, D65, D67, D69, D71, D73, D75, D77, D79, D81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

Commit message: test
Parts:
- Q1, Q3: footprint (none) -> Package_TO_SOT_SMD:SOT-23
- SW54: footprint (none) -> Rotary_Encoder:RotaryEncoder_Alps_EC11E-Switch_Vertical_H20mm_MountingHoles
Connections:
- no-connect marks 1 -> 7
Changed lines of the file:
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@@
 	)
 	(junction
-		(at 201.93 83.82)
-		(diameter 0)
-		(color 0 0 0 0)
-	)
-	(junction
 		(at 139.7 133.35)
 		(diameter 0)
@@
 	)
 	(junction
-		(at 149.86 102.87)
-		(diameter 0)
-		(color 0 0 0 0)
-	)
-	(junction
 		(at 205.74 59.69)
 		(diameter 0)
@@
 		(at 45.72 52.07)
 	)
+	(no_connect
+		(at 234.95 151.13)
+	)
+	(no_connect
+		(at 259.08 118.11)
+	)
+	(no_connect
+		(at 237.49 151.13)
+	)
+	(no_connect
+		(at 259.08 123.19)
+	)
+	(no_connect
+		(at 259.08 133.35)
+	)
+	(no_connect
+		(at 184.15 81.28)
+	)
 	(wire
 		(pts
@@
 	(wire
 		(pts
-			(xy 194.31 83.82) (xy 201.93 83.82)
-		)
-		(stroke
-			(width 0)
-			(type default)
-		)
-	)
-	(wire
-		(pts
 			(xy 36.83 26.67) (xy 36.83 36.83)
 		)
@@
 	(wire
 		(pts
-			(xy 201.93 83.82) (xy 204.47 83.82)
-		)
-		(stroke
-			(width 0)
-			(type default)
-		)
-	)
-	(wire
-		(pts
 			(xy 53.34 85.09) (xy 53.34 95.25)
 		)
@@
 	(wire
 		(pts
+			(xy 194.31 83.82) (xy 201.93 83.82)
+		)
+		(stroke
+			(width 0)
+			(type default)
+		)
+	)
+	(wire
+		(pts
 			(xy 63.5 102.87) (xy 85.09 102.87)
 		)
@@
 	(wire
 		(pts
-			(xy 149.86 102.87) (xy 151.13 102.87)
-		)
-		(stroke
-			(width 0)
-			(type default)
-		)
-	)
-	(wire
-		(pts
 			(xy 41.91 140.97) (xy 63.5 140.97)
 		)
@@
 			)
 		)
-		(property "Footprint" ""
+		(property "Footprint" "Package_TO_SOT_SMD:SOT-23"
 			(at 29.21 29.21 0)
 			(effects
@@
 			)
 		)
-		(property "Footprint" ""
+		(property "Footprint" "Package_TO_SOT_SMD:SOT-23"
 			(at 39.37 48.26 0)
 			(effects
@@
 			)
 		)
-		(property "Footprint" ""
+		(property "Footprint" "Rotary_Encoder:RotaryEncoder_Alps_EC11E-Switch_Vertical_H20mm_MountingHoles"
 			(at 152.4 183.134 0)
 			(effects

Commit message: start routing
Parts:
- removed D116: SK6812MINI, LED_SMD:LED_SK6812MINI_PLCC4_3.5x3.5mm_P1.75mm, symbol LED:SK6812MINI
- removed R5: 100kΩ, Resistor_SMD:R_0805_2012Metric, symbol Device:R
- added R3: 1kΩ, symbol Device:R
- Q1, Q3: footprint Package_TO_SOT_SMD:SOT-23 -> (none)
- R1: value 1kΩ -> 10kΩ; footprint Resistor_SMD:R_0805_2012Metric -> (none)
- renumbered SW16 to SW10, SW17 to SW11, SW18 to SW12, SW25 to SW13, SW26 to SW14, SW27 to SW15, SW28 to SW16, SW29 to SW17, SW30 to SW18, SW37 to SW19, SW3 to SW2, SW38 to SW20, SW39 to SW21, SW40 to SW22, SW41 to SW23, SW42 to SW24, SW49 to SW25, SW50 to SW26, SW51 to SW27, SW52 to SW28, SW53 to SW29, SW5 to SW3, SW7 to SW4, SW8 to SW5, SW54 to SW59, SW9 to SW6, SW13 to SW7, SW14 to SW8, SW15 to SW9
Connections:
- net COL1: now also U3.23 (P0.10-LF); no longer U3.12 (P1.06-LF)
- net COL2: now also U3.22 (P1.11-LF); no longer U3.24 (P0.09-LF)
- net COL3: now also U3.21 (P1.13-LF); no longer U3.23 (P0.10-LF)
- net COL4: now also U3.20 (P1.15-LF); no longer U3.22 (P1.11-LF)
- net COL5: now also U3.18 (P0.29-LF); no longer U3.21 (P1.13-LF)
- net COL6: now also U3.17 (P0.31-LF); no longer U3.20 (P1.15-LF)
- net LED_DAT: now also U3.2 (P0.08); no longer U3.1 (P0.06)
- net LED_PWR: now also U3.26 (P1.02-LF), R3.1; no longer R1.1, U3.2 (P0.08)
- net ROW1: now also U3.9 (P1.00); no longer U3.7 (P0.22)
- net ROW2: now also U3.10 (P0.11); no longer U3.8 (P0.24)
- net ROW3: now also U3.11 (P1.04-LF); no longer U3.9 (P1.00)
- net ROW4: now also U3.12 (P1.06-LF); no longer U3.10 (P0.11)
- net ROW5: now also U3.25 (P1.01-LF); no longer U3.11 (P1.04-LF)
- net R_E_1: now also U3.7 (P0.22); no longer U3.18 (P0.29-LF)
- net R_E_2: now also U3.8 (P0.24); no longer U3.17 (P0.31-LF)
- net R_E_S: now also U3.24 (P0.09-LF); no longer U3.27 (P1.07-LF)
- net VBAT: now also R1.1
- net at R1.2: now also Q1.1 (G), Q3.3 (D); no longer Q3.1 (G)
- net at D112.3 (DIN): now also D115.1 (DOUT)
- new net: Q3.1 (G), R3.2
- no-connect marks 7 -> 4
Other:
- moved on the sheet: D100, D103, D104, D107, D108, D111, D112, D115, D54, D61, D63, D65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

Commit message: routed about half
Parts:
- removed Q1: Q_PMOS_GSD, symbol Transistor_FET:Q_PMOS_GSD
- removed Q3: Q_NMOS_GSD, symbol Transistor_FET:Q_NMOS_GSD
- removed R1: 10kΩ, symbol Device:R
- removed R3: 1kΩ, symbol Device:R
Connections:
- net +3.3V: now also D100.4 (VDD), D103.4 (VDD), D104.4 (VDD), D107.4 (VDD), D108.4 (VDD), D111.4 (VDD), D112.4 (VDD), D115.4 (VDD), D54.4 (VDD), D61.4 (VDD), D63.4 (VDD), D65.4 (VDD), D67.4 (VDD), D69.4 (VDD), D71.4 (VDD), D73.4 (VDD), D75.4 (VDD), D77.4 (VDD), D79.4 (VDD), D81.4 (VDD), D83.4 (VDD), D85.4 (VDD), D87.4 (VDD), D89.4 (VDD), D91.4 (VDD), D93.4 (VDD), D95.4 (VDD), D97.4 (VDD), D99.4 (VDD)
- net LED_PWR: no longer names the net of U3.26 (P1.02-LF)

Commit message: renamed properly
Parts:
- renumbered D16 to D10, D17 to D11, D18 to D12, D25 to D13, D26 to D14, D27 to D15, D28 to D16, D29 to D17, D30 to D18, D37 to D19, D3 to D2, D38 to D20, D39 to D21, D40 to D22, D41 to D23, D42 to D24, D49 to D25, D50 to D26, D51 to D27, D52 to D28, D53 to D29, D5 to D3, D7 to D4, D8 to D5, D9 to D6, D13 to D7, D14 to D8, D15 to D9, D54 to L1, D77 to L10, D99 to L11, D103 to L12, D107 to L13, D111 to L14, D115 to L15, D112 to L16, D108 to L17, D104 to L18, D100 to L19, D61 to L2, D97 to L20, D95 to L21, D93 to L22, D91 to L23, D89 to L24, D87 to L25, D85 to L26, D83 to L27, D81 to L28, D79 to L29, D65 to L4, D67 to L5, D69 to L6, D71 to L7, D73 to L8, D75 to L9, D63 to l3

Commit message: placed components
Parts:
- L1, L10, L11, L12, L13, L14, L15, L16, L17, L18, L19, L2, L20, L21, L22, L23, L24, L25, L26, L27, L28, L29, L4, L5, L6, L7, L8, L9: footprint LED_SMD:LED_SK6812MINI_PLCC4_3.5x3.5mm_P1.75mm -> marbastlib-choc:LED_choc_6028R-ROT; symbol LED:SK6812MINI -> marbastlib-various:SK6812MINI-E
- L3: renamed from l3; footprint LED_SMD:LED_SK6812MINI_PLCC4_3.5x3.5mm_P1.75mm -> marbastlib-choc:LED_choc_6028R-ROT; symbol LED:SK6812MINI -> marbastlib-various:SK6812MINI-E
- SW59: footprint Rotary_Encoder:RotaryEncoder_Alps_EC11E-Switch_Vertical_H20mm_MountingHoles -> marbastlib-various:ROT_Alps_EC11E-Switch
Connections:
- net +3.3V: now also L1.1 (VDD), L10.1 (VDD), L11.1 (VDD), L12.1 (VDD), L13.1 (VDD), L14.1 (VDD), L15.1 (VDD), L16.1 (VDD), L17.1 (VDD), L18.1 (VDD), L19.1 (VDD), L2.1 (VDD), L20.1 (VDD), L21.1 (VDD), L22.1 (VDD), L23.1 (VDD), L24.1 (VDD), L25.1 (VDD), L26.1 (VDD), L27.1 (VDD), L28.1 (VDD), L29.1 (VDD), L3.1 (VDD), L4.1 (VDD), L5.1 (VDD), L6.1 (VDD), L7.1 (VDD), L8.1 (VDD), L9.1 (VDD); no longer L1.4 (VDD), L10.4 (VDD), L11.4 (VDD), L12.4 (VDD), L13.4 (VDD), L14.4 (VDD), L15.4 (VDD), L16.4 (VDD), L17.4 (VDD), L18.4 (VDD), L19.4 (VDD), L2.4 (VDD), L20.4 (VDD), L21.4 (VDD), L22.4 (VDD), L23.4 (VDD), L24.4 (VDD), L25.4 (VDD), L26.4 (VDD), L27.4 (VDD), L28.4 (VDD), L29.4 (VDD), L3.4 (VDD), L4.4 (VDD), L5.4 (VDD), L6.4 (VDD), L7.4 (VDD), L8.4 (VDD), L9.4 (VDD)
- net GND: now also L1.4 (VSS), L10.4 (VSS), L11.4 (VSS), L12.4 (VSS), L13.4 (VSS), L14.4 (VSS), L15.4 (VSS), L16.4 (VSS), L17.4 (VSS), L18.4 (VSS), L19.4 (VSS), L2.4 (VSS), L20.4 (VSS), L21.4 (VSS), L22.4 (VSS), L23.4 (VSS), L24.4 (VSS), L25.4 (VSS), L26.4 (VSS), L27.4 (VSS), L28.4 (VSS), L29.4 (VSS), L3.4 (VSS), L4.4 (VSS), L5.4 (VSS), L6.4 (VSS), L7.4 (VSS), L8.4 (VSS), L9.4 (VSS); no longer L1.2 (VSS), L10.2 (VSS), L11.2 (VSS), L12.2 (VSS), L13.2 (VSS), L14.2 (VSS), L15.2 (VSS), L16.2 (VSS), L17.2 (VSS), L18.2 (VSS), L19.2 (VSS), L2.2 (VSS), L20.2 (VSS), L21.2 (VSS), L22.2 (VSS), L23.2 (VSS), L24.2 (VSS), L25.2 (VSS), L26.2 (VSS), L27.2 (VSS), L28.2 (VSS), L29.2 (VSS), L3.2 (VSS), L4.2 (VSS), L5.2 (VSS), L6.2 (VSS), L7.2 (VSS), L8.2 (VSS), L9.2 (VSS)
- net at L19.3 (DIN): now also L18.2 (DOUT); no longer L18.1 (DOUT)
- net at L18.3 (DIN): now also L17.2 (DOUT); no longer L17.1 (DOUT)
- net at L25.3 (DIN): now also L24.2 (DOUT); no longer L24.1 (DOUT)
- net at L24.3 (DIN): now also L23.2 (DOUT); no longer L23.1 (DOUT)
- net at L3.3 (DIN): now also L2.2 (DOUT); no longer L2.1 (DOUT)
- net at L2.3 (DIN): now also L1.2 (DOUT); no longer L1.1 (DOUT)
- net at L6.3 (DIN): now also L5.2 (DOUT); no longer L5.1 (DOUT)
- net at L5.3 (DIN): now also L4.2 (DOUT); no longer L4.1 (DOUT)
- net at L12.3 (DIN): now also L11.2 (DOUT); no longer L11.1 (DOUT)
- net at L11.3 (DIN): now also L10.2 (DOUT); no longer L10.1 (DOUT)
- net at L28.3 (DIN): now also L27.2 (DOUT); no longer L27.1 (DOUT)
- net at L27.3 (DIN): now also L26.2 (DOUT); no longer L26.1 (DOUT)
- net at L10.3 (DIN): now also L9.2 (DOUT); no longer L9.1 (DOUT)
- net at L9.3 (DIN): now also L8.2 (DOUT); no longer L8.1 (DOUT)
- net at L8.3 (DIN): now also L7.2 (DOUT); no longer L7.1 (DOUT)
- net at L7.3 (DIN): now also L6.2 (DOUT); no longer L6.1 (DOUT)
- net at L14.3 (DIN): now also L13.2 (DOUT); no longer L13.1 (DOUT)
- net at L13.3 (DIN): now also L12.2 (DOUT); no longer L12.1 (DOUT)
- net at L16.3 (DIN): now also L15.2 (DOUT); no longer L15.1 (DOUT)
- net at L15.3 (DIN): now also L14.2 (DOUT); no longer L14.1 (DOUT)
- net at L29.3 (DIN): now also L28.2 (DOUT); no longer L28.1 (DOUT)
- net at L26.3 (DIN): now also L25.2 (DOUT); no longer L25.1 (DOUT)
- net at L4.3 (DIN): now also L3.2 (DOUT); no longer L3.1 (DOUT)
- net at L17.3 (DIN): now also L16.2 (DOUT); no longer L16.1 (DOUT)
- net at L23.3 (DIN): now also L22.2 (DOUT); no longer L22.1 (DOUT)
- net at L22.3 (DIN): now also L21.2 (DOUT); no longer L21.1 (DOUT)
- net at L20.3 (DIN): now also L19.2 (DOUT); no longer L19.1 (DOUT)
- net at L21.3 (DIN): now also L20.2 (DOUT); no longer L20.1 (DOUT)

Commit message: first route half
Connections:
- net COL5: now also U3.19 (P0.02-LF); no longer U3.18 (P0.29-LF)
- net COL6: now also U3.18 (P0.29-LF); no longer U3.17 (P0.31-LF)
- net ROW5: now also U3.24 (P0.09-LF); no longer U3.25 (P1.01-LF)
- net R_E_S: now also U3.17 (P0.31-LF); no longer U3.24 (P0.09-LF)
- net VBAT: now also U3.13 (BAT+)
- no-connect marks 4 -> 3
