File: keeby.kicad_pcb (KiCad board)
At the start: 2 copper layers, 66 parts, among them J1 Conn_01x04_Pin, J2 Conn_01x04_Pin, SW1 SW_Push, SW2 SW_Push, SW3 SW_Push, SW4 SW_Push, U3 SuperMini nRF52840, U4 SuperMini nRF52840

Commit message: test
Parts:
- removed D1, D10, D11, D12, D13, D14, D15, D16, D17, D18, D19, D2, D20, D21, D22, D23, D24, D25, D26, D27, D28, D29, D3, D30, D31, D32, D33, D34, D35, D36, D37, D38, D39, D4, D40, D41, D42, D43, D44, D45, D46, D47, D48, D49, D5, D50, D51, D52, D53, D55, D56, D57, D58, D59, D6, D7, D8, D9: D, Diode_SMD:D_SOD-123
- removed J1, J2: Conn_01x04_Pin, OLED-SSD1306:SSD1306-0.91-OLED-4pin-128x32
- removed U3, U4: SuperMini nRF52840, marbastlib-xp-promicroish:SuperMini_nRF52840_AH_USBup
- added SW10: SW_Push, marbastlib-choc:SW_choc_v1_HS_CPG135001S30_1u, F.Cu at (123.4, 91.7)
- added SW11: SW_Push, marbastlib-choc:SW_choc_v1_HS_CPG135001S30_1u, F.Cu at (123.4, 108.1)
- added SW12: SW_Push, marbastlib-choc:SW_choc_v1_HS_CPG135001S30_1u, F.Cu at (123.4, 124.5)
- added SW13: SW_Push, marbastlib-choc:SW_choc_v1_HS_CPG135001S30_1u, F.Cu at (141.0, 156.5)
- added SW14: SW_Push, marbastlib-choc:SW_choc_v1_HS_CPG135001S30_1u, F.Cu at (141.0, 172.9)
- added SW15: SW_Push, marbastlib-choc:SW_choc_v1_HS_CPG135001S30_1u, F.Cu at (141.0, 189.2)
- added SW16: SW_Push, marbastlib-choc:SW_choc_v1_HS_CPG135001S30_1u, F.Cu at (141.0, 205.6)
- added SW17: SW_Push, marbastlib-choc:SW_choc_v1_HS_CPG135001S30_1u, F.Cu at (141.0, 221.9)
- added SW18: SW_Push, marbastlib-choc:SW_choc_v1_HS_CPG135001S30_1u, F.Cu at (141.0, 238.3)
- added SW19: SW_Push, marbastlib-choc:SW_choc_v1_HS_CPG135001S30_1u, F.Cu at (141.0, 42.6)
- added SW20: SW_Push, marbastlib-choc:SW_choc_v1_HS_CPG135001S30_1u, F.Cu at (141.0, 59.0)
- added SW21: SW_Push, marbastlib-choc:SW_choc_v1_HS_CPG135001S30_1u, F.Cu at (141.0, 75.4)
- added SW22: SW_Push, marbastlib-choc:SW_choc_v1_HS_CPG135001S30_1u, F.Cu at (141.0, 91.7)
- added SW23: SW_Push, marbastlib-choc:SW_choc_v1_HS_CPG135001S30_1u, F.Cu at (141.0, 108.1)
- added SW24: SW_Push, marbastlib-choc:SW_choc_v1_HS_CPG135001S30_1u, F.Cu at (141.0, 124.5)
- added SW25: SW_Push, marbastlib-choc:SW_choc_v1_HS_CPG135001S30_1u, F.Cu at (158.6, 156.5)
- added SW26: SW_Push, marbastlib-choc:SW_choc_v1_HS_CPG135001S30_1u, F.Cu at (158.6, 172.9)
- added SW27: SW_Push, marbastlib-choc:SW_choc_v1_HS_CPG135001S30_1u, F.Cu at (158.6, 189.2)
- added SW28: SW_Push, marbastlib-choc:SW_choc_v1_HS_CPG135001S30_1u, F.Cu at (158.6, 205.6)
- added SW29: SW_Push, marbastlib-choc:SW_choc_v1_HS_CPG135001S30_1u, F.Cu at (158.6, 221.9)
- added SW30: SW_Push, marbastlib-choc:SW_choc_v1_HS_CPG135001S30_1u, F.Cu at (158.6, 238.3)
- added SW31: SW_Push, marbastlib-choc:SW_choc_v1_HS_CPG135001S30_1u, F.Cu at (158.6, 42.6)
- added SW32: SW_Push, marbastlib-choc:SW_choc_v1_HS_CPG135001S30_1u, F.Cu at (158.6, 59.0)
- added SW33: SW_Push, marbastlib-choc:SW_choc_v1_HS_CPG135001S30_1u, F.Cu at (158.6, 75.4)
- added SW34: SW_Push, marbastlib-choc:SW_choc_v1_HS_CPG135001S30_1u, F.Cu at (158.6, 91.7)
- added SW35: SW_Push, marbastlib-choc:SW_choc_v1_HS_CPG135001S30_1u, F.Cu at (158.6, 108.1)
- added SW36: SW_Push, marbastlib-choc:SW_choc_v1_HS_CPG135001S30_1u, F.Cu at (158.6, 124.5)
- added SW37: SW_Push, marbastlib-choc:SW_choc_v1_HS_CPG135001S30_1u, F.Cu at (176.2, 156.5)
- added SW38: SW_Push, marbastlib-choc:SW_choc_v1_HS_CPG135001S30_1u, F.Cu at (176.2, 172.9)
- added SW39: SW_Push, marbastlib-choc:SW_choc_v1_HS_CPG135001S30_1u, F.Cu at (176.2, 189.2)
- added SW40: SW_Push, marbastlib-choc:SW_choc_v1_HS_CPG135001S30_1u, F.Cu at (176.2, 205.6)
- added SW41: SW_Push, marbastlib-choc:SW_choc_v1_HS_CPG135001S30_1u, F.Cu at (176.2, 221.9)
- added SW42: SW_Push, marbastlib-choc:SW_choc_v1_HS_CPG135001S30_1u, F.Cu at (176.2, 238.3)
- added SW43: SW_Push, marbastlib-choc:SW_choc_v1_HS_CPG135001S30_1u, F.Cu at (176.2, 42.6)
- added SW44: SW_Push, marbastlib-choc:SW_choc_v1_HS_CPG135001S30_1u, F.Cu at (176.2, 59.0)
- added SW45: SW_Push, marbastlib-choc:SW_choc_v1_HS_CPG135001S30_1u, F.Cu at (176.2, 75.4)
- added SW46: SW_Push, marbastlib-choc:SW_choc_v1_HS_CPG135001S30_1u, F.Cu at (176.2, 91.7)
- added SW47: SW_Push, marbastlib-choc:SW_choc_v1_HS_CPG135001S30_1u, F.Cu at (176.2, 108.1)
- added SW48: SW_Push, marbastlib-choc:SW_choc_v1_HS_CPG135001S30_1u, F.Cu at (176.2, 124.5)
- added SW49: SW_Push, marbastlib-choc:SW_choc_v1_HS_CPG135001S30_1u, F.Cu at (193.8, 156.5)
- added SW5: SW_Push, marbastlib-choc:SW_choc_v1_HS_CPG135001S30_1u, F.Cu at (123.4, 189.2)
- added SW50: SW_Push, marbastlib-choc:SW_choc_v1_HS_CPG135001S30_1u, F.Cu at (193.8, 172.9)
- added SW51: SW_Push, marbastlib-choc:SW_choc_v1_HS_CPG135001S30_1u, F.Cu at (193.8, 189.2)
- added SW52: SW_Push, marbastlib-choc:SW_choc_v1_HS_CPG135001S30_1u, F.Cu at (193.8, 205.6)
- added SW53: SW_Push, marbastlib-choc:SW_choc_v1_HS_CPG135001S30_1u, F.Cu at (193.8, 221.9)
- added SW55: SW_Push, marbastlib-choc:SW_choc_v1_HS_CPG135001S30_1u, F.Cu at (193.8, 42.6)
- added SW56: SW_Push, marbastlib-choc:SW_choc_v1_HS_CPG135001S30_1u, F.Cu at (193.8, 59.0)
- added SW57: SW_Push, marbastlib-choc:SW_choc_v1_HS_CPG135001S30_1u, F.Cu at (193.8, 75.4)
- added SW58: SW_Push, marbastlib-choc:SW_choc_v1_HS_CPG135001S30_1u, F.Cu at (193.8, 91.7)
- added SW59: SW_Push, marbastlib-choc:SW_choc_v1_HS_CPG135001S30_1u, F.Cu at (193.8, 108.1)
- added SW6: SW_Push, marbastlib-choc:SW_choc_v1_HS_CPG135001S30_1u, F.Cu at (123.4, 75.4)
- added SW7: SW_Push, marbastlib-choc:SW_choc_v1_HS_CPG135001S30_1u, F.Cu at (123.4, 205.6)
- added SW8: SW_Push, marbastlib-choc:SW_choc_v1_HS_CPG135001S30_1u, F.Cu at (123.4, 221.9)
- added SW9: SW_Push, marbastlib-choc:SW_choc_v1_HS_CPG135001S30_1u, F.Cu at (123.4, 238.3)
- SW1, SW2, SW3, SW4: footprint marbastlib-choc:SW_choc_v1_1u -> marbastlib-choc:SW_choc_v1_HS_CPG135001S30_1u
- moved SW1 71.0 mm to (123.4, 156.5)
- moved SW3 57.9 mm to (123.4, 172.9)
- moved SW2 55.4 mm to (123.4, 42.6)
- moved SW4 54.2 mm to (123.4, 59.0)

Commit message: fix weird permission issue
Parts:
- added D1: D, Diode_SMD:D_SOD-123, F.Cu at (175.1, 215.7)
- added D10: D, Diode_SMD:D_SOD-123, F.Cu at (175.1, 111.8)
- added D100: SK6812MINI, LED_SMD:LED_SK6812MINI_PLCC4_3.5x3.5mm_P1.75mm, F.Cu at (195.7, 201.2)
- added D101: SK6812MINI, LED_SMD:LED_SK6812MINI_PLCC4_3.5x3.5mm_P1.75mm, F.Cu at (195.7, 82.2)
- added D102: SK6812MINI, LED_SMD:LED_SK6812MINI_PLCC4_3.5x3.5mm_P1.75mm, F.Cu at (195.7, 87.3)
- added D103: SK6812MINI, LED_SMD:LED_SK6812MINI_PLCC4_3.5x3.5mm_P1.75mm, F.Cu at (195.7, 206.3)
- added D104: SK6812MINI, LED_SMD:LED_SK6812MINI_PLCC4_3.5x3.5mm_P1.75mm, F.Cu at (195.7, 211.4)
- added D105: SK6812MINI, LED_SMD:LED_SK6812MINI_PLCC4_3.5x3.5mm_P1.75mm, F.Cu at (195.7, 92.4)
- added D106: SK6812MINI, LED_SMD:LED_SK6812MINI_PLCC4_3.5x3.5mm_P1.75mm, F.Cu at (195.7, 97.6)
- added D107: SK6812MINI, LED_SMD:LED_SK6812MINI_PLCC4_3.5x3.5mm_P1.75mm, F.Cu at (202.4, 185.8)
- added D108: SK6812MINI, LED_SMD:LED_SK6812MINI_PLCC4_3.5x3.5mm_P1.75mm, F.Cu at (202.4, 190.9)
- added D109: SK6812MINI, LED_SMD:LED_SK6812MINI_PLCC4_3.5x3.5mm_P1.75mm, F.Cu at (202.4, 72.0)
- added D11: D, Diode_SMD:D_SOD-123, F.Cu at (175.1, 115.2)
- added D110: SK6812MINI, LED_SMD:LED_SK6812MINI_PLCC4_3.5x3.5mm_P1.75mm, F.Cu at (202.4, 77.1)
- added D111: SK6812MINI, LED_SMD:LED_SK6812MINI_PLCC4_3.5x3.5mm_P1.75mm, F.Cu at (202.4, 196.1)
- added D112: SK6812MINI, LED_SMD:LED_SK6812MINI_PLCC4_3.5x3.5mm_P1.75mm, F.Cu at (202.4, 201.2)
- added D113: SK6812MINI, LED_SMD:LED_SK6812MINI_PLCC4_3.5x3.5mm_P1.75mm, F.Cu at (202.4, 82.2)
- added D114: SK6812MINI, LED_SMD:LED_SK6812MINI_PLCC4_3.5x3.5mm_P1.75mm, F.Cu at (202.4, 87.3)
- added D115: SK6812MINI, LED_SMD:LED_SK6812MINI_PLCC4_3.5x3.5mm_P1.75mm, F.Cu at (202.4, 206.3)
- added D116: SK6812MINI, LED_SMD:LED_SK6812MINI_PLCC4_3.5x3.5mm_P1.75mm, F.Cu at (202.4, 211.4)
- added D117: SK6812MINI, LED_SMD:LED_SK6812MINI_PLCC4_3.5x3.5mm_P1.75mm, F.Cu at (202.4, 92.4)
- added D118: SK6812MINI, LED_SMD:LED_SK6812MINI_PLCC4_3.5x3.5mm_P1.75mm, F.Cu at (202.4, 97.6)
- added D12: D, Diode_SMD:D_SOD-123, F.Cu at (175.1, 118.5)
- added D13: D, Diode_SMD:D_SOD-123, F.Cu at (175.1, 235.8)
- added D14: D, Diode_SMD:D_SOD-123, F.Cu at (175.1, 239.1)
- added D15: D, Diode_SMD:D_SOD-123, F.Cu at (180.9, 215.7)
- added D16: D, Diode_SMD:D_SOD-123, F.Cu at (180.9, 219.0)
- added D17: D, Diode_SMD:D_SOD-123, F.Cu at (180.9, 222.4)
- added D18: D, Diode_SMD:D_SOD-123, F.Cu at (180.9, 225.7)
- added D19: D, Diode_SMD:D_SOD-123, F.Cu at (175.1, 121.9)
- added D2: D, Diode_SMD:D_SOD-123, F.Cu at (175.1, 101.8)
- added D20: D, Diode_SMD:D_SOD-123, F.Cu at (175.1, 125.2)
- added D21: D, Diode_SMD:D_SOD-123, F.Cu at (180.9, 101.8)
- added D22: D, Diode_SMD:D_SOD-123, F.Cu at (180.9, 105.1)
- added D23: D, Diode_SMD:D_SOD-123, F.Cu at (180.9, 108.5)
- added D24: D, Diode_SMD:D_SOD-123, F.Cu at (180.9, 111.8)
- added D25: D, Diode_SMD:D_SOD-123, F.Cu at (180.9, 229.1)
- added D26: D, Diode_SMD:D_SOD-123, F.Cu at (180.9, 232.4)
- added D27: D, Diode_SMD:D_SOD-123, F.Cu at (180.9, 235.8)
- added D28: D, Diode_SMD:D_SOD-123, F.Cu at (180.9, 239.1)
- added D29: D, Diode_SMD:D_SOD-123, F.Cu at (186.7, 215.7)
- added D3: D, Diode_SMD:D_SOD-123, F.Cu at (175.1, 219.0)
- added D30: D, Diode_SMD:D_SOD-123, F.Cu at (186.7, 219.0)
- added D31: D, Diode_SMD:D_SOD-123, F.Cu at (180.9, 115.2)
- added D32: D, Diode_SMD:D_SOD-123, F.Cu at (180.9, 118.5)
- added D33: D, Diode_SMD:D_SOD-123, F.Cu at (180.9, 121.9)
- added D34: D, Diode_SMD:D_SOD-123, F.Cu at (180.9, 125.2)
- added D35: D, Diode_SMD:D_SOD-123, F.Cu at (186.7, 101.8)
- added D36: D, Diode_SMD:D_SOD-123, F.Cu at (186.7, 105.1)
- added D37: D, Diode_SMD:D_SOD-123, F.Cu at (186.7, 222.4)
- added D38: D, Diode_SMD:D_SOD-123, F.Cu at (186.7, 225.7)
- added D39: D, Diode_SMD:D_SOD-123, F.Cu at (186.7, 229.1)
- added D4: D, Diode_SMD:D_SOD-123, F.Cu at (175.1, 105.1)
- added D40: D, Diode_SMD:D_SOD-123, F.Cu at (186.7, 232.4)
- added D41: D, Diode_SMD:D_SOD-123, F.Cu at (186.7, 235.8)
- added D42: D, Diode_SMD:D_SOD-123, F.Cu at (186.7, 239.1)
- added D43: D, Diode_SMD:D_SOD-123, F.Cu at (186.7, 108.5)
- added D44: D, Diode_SMD:D_SOD-123, F.Cu at (186.7, 111.8)
- added D45: D, Diode_SMD:D_SOD-123, F.Cu at (186.7, 115.2)
- added D46: D, Diode_SMD:D_SOD-123, F.Cu at (186.7, 118.5)
- added D47: D, Diode_SMD:D_SOD-123, F.Cu at (186.7, 121.9)
- added D48: D, Diode_SMD:D_SOD-123, F.Cu at (186.7, 125.2)
- added D49: D, Diode_SMD:D_SOD-123, F.Cu at (192.5, 215.7)
- added D5: D, Diode_SMD:D_SOD-123, F.Cu at (175.1, 222.4)
- added D50: D, Diode_SMD:D_SOD-123, F.Cu at (192.5, 219.0)
- added D51: D, Diode_SMD:D_SOD-123, F.Cu at (192.5, 222.4)
- added D52: D, Diode_SMD:D_SOD-123, F.Cu at (192.5, 225.7)
- added D53: D, Diode_SMD:D_SOD-123, F.Cu at (192.5, 229.1)
- added D54: SK6812MINI, LED_SMD:LED_SK6812MINI_PLCC4_3.5x3.5mm_P1.75mm, F.Cu at (175.5, 185.8)
- added D55: D, Diode_SMD:D_SOD-123, F.Cu at (192.5, 101.8)
- added D56: D, Diode_SMD:D_SOD-123, F.Cu at (192.5, 105.1)
- added D57: D, Diode_SMD:D_SOD-123, F.Cu at (192.5, 108.5)
- added D58: D, Diode_SMD:D_SOD-123, F.Cu at (192.5, 111.8)
- added D59: D, Diode_SMD:D_SOD-123, F.Cu at (192.5, 115.2)
- added D6: D, Diode_SMD:D_SOD-123, F.Cu at (175.1, 108.5)
- added D60: SK6812MINI, LED_SMD:LED_SK6812MINI_PLCC4_3.5x3.5mm_P1.75mm, F.Cu at (175.5, 72.0)
- added D61: SK6812MINI, LED_SMD:LED_SK6812MINI_PLCC4_3.5x3.5mm_P1.75mm, F.Cu at (175.5, 190.9)
- added D62: SK6812MINI, LED_SMD:LED_SK6812MINI_PLCC4_3.5x3.5mm_P1.75mm, F.Cu at (175.5, 77.1)
- added D63: SK6812MINI, LED_SMD:LED_SK6812MINI_PLCC4_3.5x3.5mm_P1.75mm, F.Cu at (175.5, 196.1)
- added D64: SK6812MINI, LED_SMD:LED_SK6812MINI_PLCC4_3.5x3.5mm_P1.75mm, F.Cu at (175.5, 82.2)
- added D65: SK6812MINI, LED_SMD:LED_SK6812MINI_PLCC4_3.5x3.5mm_P1.75mm, F.Cu at (175.5, 201.2)
- added D66: SK6812MINI, LED_SMD:LED_SK6812MINI_PLCC4_3.5x3.5mm_P1.75mm, F.Cu at (175.5, 87.3)
- added D67: SK6812MINI, LED_SMD:LED_SK6812MINI_PLCC4_3.5x3.5mm_P1.75mm, F.Cu at (175.5, 206.3)
- added D68: SK6812MINI, LED_SMD:LED_SK6812MINI_PLCC4_3.5x3.5mm_P1.75mm, F.Cu at (175.5, 92.4)
- added D69: SK6812MINI, LED_SMD:LED_SK6812MINI_PLCC4_3.5x3.5mm_P1.75mm, F.Cu at (175.5, 211.4)
- added D7: D, Diode_SMD:D_SOD-123, F.Cu at (175.1, 225.7)
- added D70: SK6812MINI, LED_SMD:LED_SK6812MINI_PLCC4_3.5x3.5mm_P1.75mm, F.Cu at (175.5, 97.6)
- added D71: SK6812MINI, LED_SMD:LED_SK6812MINI_PLCC4_3.5x3.5mm_P1.75mm, F.Cu at (182.2, 185.8)
- added D72: SK6812MINI, LED_SMD:LED_SK6812MINI_PLCC4_3.5x3.5mm_P1.75mm, F.Cu at (182.2, 72.0)
- added D73: SK6812MINI, LED_SMD:LED_SK6812MINI_PLCC4_3.5x3.5mm_P1.75mm, F.Cu at (182.2, 190.9)
- added D74: SK6812MINI, LED_SMD:LED_SK6812MINI_PLCC4_3.5x3.5mm_P1.75mm, F.Cu at (182.2, 77.1)
- added D75: SK6812MINI, LED_SMD:LED_SK6812MINI_PLCC4_3.5x3.5mm_P1.75mm, F.Cu at (182.2, 196.1)
- added D76: SK6812MINI, LED_SMD:LED_SK6812MINI_PLCC4_3.5x3.5mm_P1.75mm, F.Cu at (182.2, 82.2)
- added D77: SK6812MINI, LED_SMD:LED_SK6812MINI_PLCC4_3.5x3.5mm_P1.75mm, F.Cu at (182.2, 201.2)
- added D78: SK6812MINI, LED_SMD:LED_SK6812MINI_PLCC4_3.5x3.5mm_P1.75mm, F.Cu at (182.2, 87.3)
- added D79: SK6812MINI, LED_SMD:LED_SK6812MINI_PLCC4_3.5x3.5mm_P1.75mm, F.Cu at (182.2, 206.3)
- added D8: D, Diode_SMD:D_SOD-123, F.Cu at (175.1, 229.1)
- added D80: SK6812MINI, LED_SMD:LED_SK6812MINI_PLCC4_3.5x3.5mm_P1.75mm, F.Cu at (182.2, 92.4)
- added D81: SK6812MINI, LED_SMD:LED_SK6812MINI_PLCC4_3.5x3.5mm_P1.75mm, F.Cu at (182.2, 211.4)
- added D82: SK6812MINI, LED_SMD:LED_SK6812MINI_PLCC4_3.5x3.5mm_P1.75mm, F.Cu at (182.2, 97.6)
- added D83: SK6812MINI, LED_SMD:LED_SK6812MINI_PLCC4_3.5x3.5mm_P1.75mm, F.Cu at (188.9, 185.8)
- added D84: SK6812MINI, LED_SMD:LED_SK6812MINI_PLCC4_3.5x3.5mm_P1.75mm, F.Cu at (188.9, 72.0)
- added D85: SK6812MINI, LED_SMD:LED_SK6812MINI_PLCC4_3.5x3.5mm_P1.75mm, F.Cu at (188.9, 190.9)
- added D86: SK6812MINI, LED_SMD:LED_SK6812MINI_PLCC4_3.5x3.5mm_P1.75mm, F.Cu at (188.9, 77.1)
- added D87: SK6812MINI, LED_SMD:LED_SK6812MINI_PLCC4_3.5x3.5mm_P1.75mm, F.Cu at (188.9, 196.1)
- added D88: SK6812MINI, LED_SMD:LED_SK6812MINI_PLCC4_3.5x3.5mm_P1.75mm, F.Cu at (188.9, 82.2)
- added D89: SK6812MINI, LED_SMD:LED_SK6812MINI_PLCC4_3.5x3.5mm_P1.75mm, F.Cu at (188.9, 201.2)
- added D9: D, Diode_SMD:D_SOD-123, F.Cu at (175.1, 232.4)
- added D90: SK6812MINI, LED_SMD:LED_SK6812MINI_PLCC4_3.5x3.5mm_P1.75mm, F.Cu at (188.9, 87.3)
- added D91: SK6812MINI, LED_SMD:LED_SK6812MINI_PLCC4_3.5x3.5mm_P1.75mm, F.Cu at (188.9, 206.3)
- added D92: SK6812MINI, LED_SMD:LED_SK6812MINI_PLCC4_3.5x3.5mm_P1.75mm, F.Cu at (188.9, 92.4)
- added D93: SK6812MINI, LED_SMD:LED_SK6812MINI_PLCC4_3.5x3.5mm_P1.75mm, F.Cu at (188.9, 211.4)
- added D94: SK6812MINI, LED_SMD:LED_SK6812MINI_PLCC4_3.5x3.5mm_P1.75mm, F.Cu at (188.9, 97.6)
- added D95: SK6812MINI, LED_SMD:LED_SK6812MINI_PLCC4_3.5x3.5mm_P1.75mm, F.Cu at (195.7, 185.8)
- added D96: SK6812MINI, LED_SMD:LED_SK6812MINI_PLCC4_3.5x3.5mm_P1.75mm, F.Cu at (195.7, 72.0)
- added D97: SK6812MINI, LED_SMD:LED_SK6812MINI_PLCC4_3.5x3.5mm_P1.75mm, F.Cu at (195.7, 190.9)
- added D98: SK6812MINI, LED_SMD:LED_SK6812MINI_PLCC4_3.5x3.5mm_P1.75mm, F.Cu at (195.7, 77.1)
- added D99: SK6812MINI, LED_SMD:LED_SK6812MINI_PLCC4_3.5x3.5mm_P1.75mm, F.Cu at (195.7, 196.1)
- added H1: MountingHole, MountingHole:MountingHole_2.1mm, F.Cu at (198.2, 216.9)
- added H2: MountingHole, MountingHole:MountingHole_2.1mm, F.Cu at (198.2, 103.0)
- added H3: MountingHole, MountingHole:MountingHole_2.1mm, F.Cu at (198.2, 222.6)
- added H4: MountingHole, MountingHole:MountingHole_2.1mm, F.Cu at (198.2, 108.7)
- added H5: MountingHole, MountingHole:MountingHole_2.1mm, F.Cu at (198.2, 228.4)
- added H6: MountingHole, MountingHole:MountingHole_2.1mm, F.Cu at (198.2, 114.5)
- added H7: MountingHole, MountingHole:MountingHole_2.1mm, F.Cu at (198.2, 234.1)
- added H8: MountingHole, MountingHole:MountingHole_2.1mm, F.Cu at (198.2, 120.2)
- added J1: Conn_01x04_Pin, OLED-SSD1306:SSD1306-0.91-OLED-4pin-128x32, F.Cu at (208.5, 160.2)
- added J2: Conn_01x04_Pin, OLED-SSD1306:SSD1306-0.91-OLED-4pin-128x32, F.Cu at (208.5, 144.9)
- added J3: JST_PH, Connector_JST:JST_PH_S2B-PH-K_1x02_P2.00mm_Horizontal, F.Cu at (87.2, 244.7)
- added J4: JST_PH, Connector_JST:JST_PH_S2B-PH-K_1x02_P2.00mm_Horizontal, F.Cu at (87.2, 130.8)
- added Q1: Q_PMOS_GSD, Package_TO_SOT_SMD:SOT-23, F.Cu at (94.6, 244.6)
- added Q2: Q_PMOS_GSD, Package_TO_SOT_SMD:SOT-23, F.Cu at (94.6, 130.7)
- added Q3: Q_NMOS_GSD, Package_TO_SOT_SMD:SOT-23, F.Cu at (94.6, 249.0)
- added Q4: Q_NMOS_GSD, Package_TO_SOT_SMD:SOT-23, F.Cu at (94.6, 135.1)
- added R1: 1kΩ, Resistor_SMD:R_0805_2012Metric, F.Cu at (99.2, 243.8)
- added R2: 1kΩ, Resistor_SMD:R_0805_2012Metric, F.Cu at (99.2, 129.9)
- added R5: 100kΩ, Resistor_SMD:R_0805_2012Metric, F.Cu at (99.2, 246.8)
- added R6: 100kΩ, Resistor_SMD:R_0805_2012Metric, F.Cu at (99.2, 132.9)
- added SW54: RotaryEncoder_Switch, Rotary_Encoder:RotaryEncoder_Alps_EC11E-Switch_Vertical_H20mm_MountingHoles, F.Cu at (174.2, 245.9)
- added SW60: RotaryEncoder_Switch, Rotary_Encoder:RotaryEncoder_Alps_EC11E-Switch_Vertical_H20mm_MountingHoles, F.Cu at (174.2, 132.0)
- added SW61: SW_SPDT, Button_Switch_SMD:SW_SPDT_PCM12, F.Cu at (195.6, 243.8)
- added SW62: SW_SPDT, Button_Switch_SMD:SW_SPDT_PCM12, F.Cu at (195.6, 129.9)
- added U3: SuperMini nRF52840, marbastlib-xp-promicroish:SuperMini_nRF52840_AH_USBup, F.Cu at (186.5, 162.5)
- added U4: SuperMini nRF52840, marbastlib-xp-promicroish:SuperMini_nRF52840_AH_USBup, F.Cu at (186.5, 48.7)
- moved SW1 32.1 mm to (91.7, 151.7)
- moved SW10 32.1 mm to (91.7, 86.9)
- moved SW11 32.1 mm to (91.7, 103.3)
- moved SW12 32.1 mm to (91.7, 119.6)
- moved SW13 32.1 mm to (109.3, 151.7)
- moved SW14 32.1 mm to (109.3, 168.1)
- moved SW15 32.1 mm to (109.3, 184.4)
- moved SW16 32.1 mm to (109.3, 200.8)
- moved SW17 32.1 mm to (109.3, 217.1)
- moved SW18 32.1 mm to (109.3, 233.5)
- moved SW19 32.1 mm to (109.3, 37.8)
- moved SW2 32.1 mm to (91.7, 37.8)
- moved SW20 32.1 mm to (109.3, 54.2)
- moved SW21 32.1 mm to (109.3, 70.6)
- moved SW22 32.1 mm to (109.3, 86.9)
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
Commit message: start routing
Parts:
- removed D116, D118: SK6812MINI, LED_SMD:LED_SK6812MINI_PLCC4_3.5x3.5mm_P1.75mm
- removed Q1, Q2: Q_PMOS_GSD, Package_TO_SOT_SMD:SOT-23
- removed Q3, Q4: Q_NMOS_GSD, Package_TO_SOT_SMD:SOT-23
- removed R1, R2: 1kΩ, Resistor_SMD:R_0805_2012Metric
- removed R5, R6: 100kΩ, Resistor_SMD:R_0805_2012Metric
- D1, D10, D11, D12, D13, D14, D15, D16, D17, D18, D19, D2, D20, D21, D22, D23, D24, D25, D26, D27, D28, D29, D3, D30, D31, D32, D33, D34, D35, D36, D37, D38, D39, D4, D40, D41, D42, D43, D44, D45, D46, D47, D48, D49, D5, D50, D51, D52, D53, D55, D56, D57, D58, D59, D6, D7, D8, D9: moved to B.Cu
- SW54: value RotaryEncoder_Switch -> SW_Push; footprint Rotary_Encoder:RotaryEncoder_Alps_EC11E-Switch_Vertical_H20mm_MountingHoles -> marbastlib-choc:SW_choc_v1_HS_CPG135001S30_1u
- SW59: value SW_Push -> RotaryEncoder_Switch; footprint marbastlib-choc:SW_choc_v1_HS_CPG135001S30_1u -> Rotary_Encoder:RotaryEncoder_Alps_EC11E-Switch_Vertical_H20mm_MountingHoles
- moved D13 225.9 mm to (29.8, 62.9), turned to -90 degrees
- moved D1 225.0 mm to (29.8, 43.8), turned to -90 degrees
- moved SW41 222.5 mm to (304.8, 62.9)
- moved D14 216.8 mm to (48.8, 62.9), turned to -90 degrees
- moved D3 216.0 mm to (48.8, 43.8), turned to -90 degrees
- moved D25 210.9 mm to (29.8, 81.9), turned to -90 degrees
- moved D5 210.7 mm to (67.8, 41.0), turned to -90 degrees
- moved D7 207.3 mm to (86.9, 38.1), turned to -90 degrees
- moved SW30 206.9 mm to (209.6, 43.8)
- moved D8 200.4 mm to (106.0, 41.0), turned to -90 degrees
- moved D26 200.2 mm to (48.8, 81.9), turned to -90 degrees
- moved D37 198.4 mm to (29.8, 101.0), turned to -90 degrees
- moved J4 197.8 mm to (223.5, 274.1), turned to 90 degrees
- moved SW40 197.4 mm to (285.8, 62.9)
- moved D9 195.1 mm to (125.0, 43.8), turned to -90 degrees
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Connections:
- D115 pad 1: Net-(D115-DOUT) -> Net-(D112-DIN)
- D117 pad 1: Net-(D117-DOUT) -> Net-(D114-DIN)
- SW10 pad 2: Net-(D10-A) -> Net-(D16-A)
- SW11 pad 2: Net-(D11-A) -> Net-(D17-A)
- SW12 pad 2: Net-(D12-A) -> Net-(D18-A)
- SW13 pad 2: Net-(D13-A) -> Net-(D25-A)
- SW14 pad 2: Net-(D14-A) -> Net-(D26-A)
- SW15 pad 2: Net-(D15-A) -> Net-(D27-A)
- SW16 pad 2: Net-(D16-A) -> Net-(D28-A)
- SW17 pad 2: Net-(D17-A) -> Net-(D29-A)
- SW18 pad 2: Net-(D18-A) -> Net-(D30-A)
- SW19 pad 2: Net-(D19-A) -> Net-(D37-A)
- SW2 pad 1: COL1 -> COL2
- SW2 pad 2: Net-(D2-A) -> Net-(D3-A)
- SW20 pad 2: Net-(D20-A) -> Net-(D38-A)
- SW21 pad 2: Net-(D21-A) -> Net-(D39-A)
- SW22 pad 2: Net-(D22-A) -> Net-(D40-A)
- SW23 pad 2: Net-(D23-A) -> Net-(D41-A)
- SW24 pad 2: Net-(D24-A) -> Net-(D42-A)
- SW25 pad 2: Net-(D25-A) -> Net-(D49-A)
- SW26 pad 2: Net-(D26-A) -> Net-(D50-A)
- SW27 pad 2: Net-(D27-A) -> Net-(D51-A)
- SW28 pad 2: Net-(D28-A) -> Net-(D52-A)
- SW29 pad 2: Net-(D29-A) -> Net-(D53-A)
- SW3 pad 1: COL2 -> COL3
- SW3 pad 2: Net-(D3-A) -> Net-(D5-A)
- SW30 pad 1: COL6 -> COL1
- SW30 pad 2: Net-(D30-A) -> Net-(D2-A)
- SW31 pad 1: COL1 -> COL2
- SW31 pad 2: Net-(D31-A) -> Net-(D4-A)
- SW32 pad 1: COL2 -> COL3
- SW32 pad 2: Net-(D32-A) -> Net-(D6-A)
- SW33 pad 1: COL3 -> COL4
- SW33 pad 2: Net-(D33-A) -> Net-(D10-A)
- SW34 pad 1: COL4 -> COL5
- SW34 pad 2: Net-(D34-A) -> Net-(D11-A)
- SW35 pad 1: COL5 -> COL6
- SW35 pad 2: Net-(D35-A) -> Net-(D12-A)
- SW36 pad 1: COL6 -> COL1
- SW36 pad 2: Net-(D36-A) -> Net-(D19-A)
- SW37 pad 1: COL1 -> COL2
- SW37 pad 2: Net-(D37-A) -> Net-(D20-A)
- SW38 pad 1: COL2 -> COL3
- SW38 pad 2: Net-(D38-A) -> Net-(D21-A)
- SW39 pad 1: COL3 -> COL4
- SW39 pad 2: Net-(D39-A) -> Net-(D22-A)
- SW4 pad 1: COL2 -> COL4
- SW4 pad 2: Net-(D4-A) -> Net-(D7-A)
- SW40 pad 1: COL4 -> COL5
- SW40 pad 2: Net-(D40-A) -> Net-(D23-A)
- SW41 pad 1: COL5 -> COL6
- SW41 pad 2: Net-(D41-A) -> Net-(D24-A)
- SW42 pad 1: COL6 -> COL1
- SW42 pad 2: Net-(D42-A) -> Net-(D31-A)
- SW43 pad 1: COL1 -> COL2
- SW43 pad 2: Net-(D43-A) -> Net-(D32-A)
- SW44 pad 1: COL2 -> COL3
- SW44 pad 2: Net-(D44-A) -> Net-(D33-A)
- SW45 pad 1: COL3 -> COL4
- SW45 pad 2: Net-(D45-A) -> Net-(D34-A)
- SW46 pad 1: COL4 -> COL5
- SW46 pad 2: Net-(D46-A) -> Net-(D35-A)
- SW47 pad 1: COL5 -> COL6
- SW47 pad 2: Net-(D47-A) -> Net-(D36-A)
- SW48 pad 1: COL6 -> COL1
- SW48 pad 2: Net-(D48-A) -> Net-(D43-A)
- SW49 pad 1: COL1 -> COL2
- SW49 pad 2: Net-(D49-A) -> Net-(D44-A)
- SW5 pad 1: COL3 -> COL5
- SW5 pad 2: Net-(D5-A) -> Net-(D8-A)
- SW50 pad 1: COL2 -> COL3
- SW50 pad 2: Net-(D50-A) -> Net-(D45-A)
- SW51 pad 1: COL3 -> COL4
- SW51 pad 2: Net-(D51-A) -> Net-(D46-A)
- SW52 pad 1: COL4 -> COL5
- SW52 pad 2: Net-(D52-A) -> Net-(D47-A)
- SW53 pad 1: COL5 -> COL6
- SW53 pad 2: Net-(D53-A) -> Net-(D48-A)
- SW55 pad 1: COL1 -> COL2
- SW55 pad 2: Net-(D55-A) -> Net-(D56-A)
- SW56 pad 1: COL2 -> COL3
- SW56 pad 2: Net-(D56-A) -> Net-(D57-A)
- SW57 pad 1: COL3 -> COL4
- SW57 pad 2: Net-(D57-A) -> Net-(D58-A)
- SW58 pad 1: COL4 -> COL5
- SW58 pad 2: Net-(D58-A) -> Net-(D59-A)
- SW6 pad 1: COL3 -> COL6
- SW6 pad 2: Net-(D6-A) -> Net-(D9-A)
- SW7 pad 1: COL4 -> COL1
- SW7 pad 2: Net-(D7-A) -> Net-(D13-A)
- SW8 pad 1: COL5 -> COL2
- SW8 pad 2: Net-(D8-A) -> Net-(D14-A)
- SW9 pad 1: COL6 -> COL3
- SW9 pad 2: Net-(D9-A) -> Net-(D15-A)
- U3 pad 1: LED_DAT -> unconnected-(U3-P0.06-Pad1)
- U3 pad 10: ROW4 -> ROW2
- U3 pad 11: ROW5 -> ROW3
- U3 pad 12: COL1 -> ROW4
- U3 pad 17: R_E_2 -> COL6
- U3 pad 18: R_E_1 -> COL5
- U3 pad 2: LED_PWR -> LED_DAT
- U3 pad 20: COL6 -> COL4
- U3 pad 21: COL5 -> COL3
- U3 pad 22: COL4 -> COL2
- U3 pad 23: COL3 -> COL1
- U3 pad 24: COL2 -> R_E_S
- U3 pad 25: unconnected-(U3-P1.01-LF-Pad25) -> ROW5
- U3 pad 26: unconnected-(U3-P1.02-LF-Pad26) -> LED_PWR
- U3 pad 27: R_E_S -> unconnected-(U3-P1.07-LF-Pad27)
- U3 pad 7: ROW1 -> R_E_1
- U3 pad 8: ROW2 -> R_E_2
- U3 pad 9: ROW3 -> ROW1
- U4 pad 1: LED_DAT -> unconnected-(U4-P0.06-Pad1)
- U4 pad 10: ROW4 -> ROW2
- U4 pad 11: ROW5 -> ROW3
- U4 pad 12: COL1 -> ROW4
- U4 pad 17: R_E_2 -> COL6
- U4 pad 18: R_E_1 -> COL5
- U4 pad 2: LED_PWR -> LED_DAT
- U4 pad 20: COL6 -> COL4
- U4 pad 21: COL5 -> COL3
- U4 pad 22: COL4 -> COL2
- U4 pad 23: COL3 -> COL1
- U4 pad 24: COL2 -> R_E_S
- U4 pad 25: unconnected-(U4-P1.01-LF-Pad25) -> ROW5
- U4 pad 26: unconnected-(U4-P1.02-LF-Pad26) -> LED_PWR
- U4 pad 27: R_E_S -> unconnected-(U4-P1.07-LF-Pad27)
- U4 pad 7: ROW1 -> R_E_1
- U4 pad 8: ROW2 -> R_E_2
- U4 pad 9: ROW3 -> ROW1
Routing:
- net Net-(D48-A): track 0.00 -> 10.1 mm
- net Net-(D47-A): track 0.00 -> 10.1 mm
- net Net-(D43-A): track 0.00 -> 10.1 mm
- net Net-(D57-A): track 0.00 -> 10.1 mm
- net Net-(D36-A): track 0.00 -> 10.1 mm
- net Net-(D35-A): track 0.00 -> 10.1 mm
- net Net-(D31-A): track 0.00 -> 10.1 mm
- net Net-(D24-A): track 0.00 -> 10.1 mm
- net Net-(D23-A): track 0.00 -> 10.1 mm
- net Net-(D2-A): track 0.00 -> 10.1 mm
- net Net-(D19-A): track 0.00 -> 10.1 mm
- net Net-(D12-A): track 0.00 -> 10.1 mm
- net Net-(D11-A): track 0.00 -> 10.1 mm
- net Net-(D37-A): track 0.00 -> 10.1 mm
- net Net-(D44-A): track 0.00 -> 10.1 mm
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Other:
- board outline added: 288 x 117.5 mm

Commit message: routed about half
Parts:
- removed D10, D11, D12, D19, D2, D20, D21, D22, D23, D24, D31, D32, D33, D34, D35, D36, D4, D43, D44, D45, D46, D47, D48, D55, D56, D57, D58, D59, D6: D, Diode_SMD:D_SOD-123
- removed D101, D102, D105, D106, D109, D110, D113, D114, D117, D60, D62, D64, D66, D68, D70, D72, D74, D76, D78, D80, D82, D84, D86, D88, D90, D92, D94, D96, D98: SK6812MINI, LED_SMD:LED_SK6812MINI_PLCC4_3.5x3.5mm_P1.75mm
- removed H2, H4, H6, H8: MountingHole, MountingHole:MountingHole_2.1mm
- removed J2: Conn_01x04_Pin, OLED-SSD1306:SSD1306-0.91-OLED-4pin-128x32
- removed J4: JST_PH, Connector_JST:JST_PH_S2B-PH-K_1x02_P2.00mm_Horizontal
- removed SW30, SW31, SW32, SW33, SW34, SW35, SW36, SW37, SW38, SW39, SW40, SW41, SW42, SW43, SW44, SW45, SW46, SW47, SW48, SW49, SW50, SW51, SW52, SW53, SW54, SW55, SW56, SW57, SW58: SW_Push, marbastlib-choc:SW_choc_v1_HS_CPG135001S30_1u
- removed SW60: RotaryEncoder_Switch, Rotary_Encoder:RotaryEncoder_Alps_EC11E-Switch_Vertical_H20mm_MountingHoles
- removed SW62: SW_SPDT, Button_Switch_SMD:SW_SPDT_PCM12
- removed U4: SuperMini nRF52840, marbastlib-xp-promicroish:SuperMini_nRF52840_AH_USBup
- moved J3 228.6 mm to (151.6, 85.0)
- moved H7 223.4 mm to (45.4, 146.0), turned to -90 degrees
- moved H5 212.3 mm to (51.4, 146.0), turned to -90 degrees
- moved H3 202.2 mm to (56.4, 146.0), turned to -90 degrees
- moved J1 199.2 mm to (162.9, 35.1), turned to -90 degrees
- moved H1 191.3 mm to (62.4, 146.0), turned to -90 degrees
- moved SW61 182.1 mm to (163.7, 85.5)
- moved D54 156.9 mm to (133.0, 39.0), turned to 0 degrees
- moved D61 149.5 mm to (114.0, 36.0), turned to 0 degrees
- moved D63 144.2 mm to (95.0, 33.0), turned to 0 degrees
- moved D65 135.3 mm to (76.2, 36.1), turned to 0 degrees
- moved D107 131.8 mm to (133.0, 77.0), turned to 0 degrees
- moved D75 131.7 mm to (76.0, 55.0)
- moved D77 131.4 mm to (95.0, 52.0)
- moved D67 129.4 mm to (57.2, 38.9), turned to 0 degrees
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Routing:
- net Net-(J3-Pin_1): track 0.00 -> 10.8 mm
- net Net-(D48-A): track 10.1 -> 0.00 mm
- net Net-(D47-A): track 10.1 -> 0.00 mm
- net Net-(D43-A): track 10.1 -> 0.00 mm
- net Net-(D57-A): track 10.1 -> 0.00 mm
- net Net-(D36-A): track 10.1 -> 0.00 mm
- net Net-(D35-A): track 10.1 -> 0.00 mm
- net Net-(D31-A): track 10.1 -> 0.00 mm
- net Net-(D24-A): track 10.1 -> 0.00 mm
- net Net-(D23-A): track 10.1 -> 0.00 mm
- net Net-(D2-A): track 10.1 -> 0.00 mm
- net Net-(D19-A): track 10.1 -> 0.00 mm
- net Net-(D12-A): track 10.1 -> 0.00 mm
- net Net-(D11-A): track 10.1 -> 0.00 mm
- net Net-(D44-A): track 10.1 -> 0.00 mm
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Other:
- board size 288 x 117.5 mm -> 143 x 117 mm
