File: keeby.kicad_pcb (KiCad board)
At the start: 2 copper layers, 143 x 117 mm, 96 parts, among them J1 Conn_01x04_Pin, J3 JST_PH, SW1 SW_Push, SW10 SW_Push, SW11 SW_Push, SW12 SW_Push, SW13 SW_Push, SW14 SW_Push, SW15 SW_Push, SW16 SW_Push, SW17 SW_Push, SW18 SW_Push, SW19 SW_Push, SW2 SW_Push, SW20 SW_Push, SW21 SW_Push, SW22 SW_Push, SW23 SW_Push, SW24 SW_Push, SW25 SW_Push, SW26 SW_Push, SW27 SW_Push, SW28 SW_Push, SW29 SW_Push, SW3 SW_Push, SW4 SW_Push, SW5 SW_Push, SW59 RotaryEncoder_Switch, SW6 SW_Push, SW61 SW_SPDT, SW7 SW_Push, SW8 SW_Push, SW9 SW_Push, U3 SuperMini nRF52840

Commit message: renamed properly
Other:
- board size 143 x 117 mm -> 380 x 251 mm
Changed lines of the file:
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@@
 	(net 81 "VBAT")
 	(net 82 "unconnected-(U3-P1.07-LF-Pad27)")
-	(net 83 "LED_PWR")
-	(net 84 "unconnected-(U3-P0.06-Pad1)")
-	(net 85 "unconnected-(U3-BAT+-Pad13)")
-	(net 86 "unconnected-(U3-RST-Pad15)")
-	(net 87 "unconnected-(U3-P0.02-LF-Pad19)")
+	(net 83 "unconnected-(U3-P0.06-Pad1)")
+	(net 84 "unconnected-(U3-BAT+-Pad13)")
+	(net 85 "unconnected-(U3-RST-Pad15)")
+	(net 86 "unconnected-(U3-P0.02-LF-Pad19)")
+	(net 87 "LED_PWR")
 	(footprint "marbastlib-choc:SW_choc_v1_HS_CPG135001S30_1u"
 		(layer "F.Cu")
@@
 			(layers "*.Cu" "B.Mask")
 			(remove_unused_layers no)
-			(net 84 "unconnected-(U3-P0.06-Pad1)")
+			(net 83 "unconnected-(U3-P0.06-Pad1)")
 			(pinfunction "P0.06")
 			(pintype "bidirectional")
@@
 			(layers "*.Cu" "B.Mask")
 			(remove_unused_layers no)
-			(net 85 "unconnected-(U3-BAT+-Pad13)")
+			(net 84 "unconnected-(U3-BAT+-Pad13)")
 			(pinfunction "BAT+")
 			(pintype "power_in+no_connect")
@@
 			(layers "*.Cu" "B.Mask")
 			(remove_unused_layers no)
-			(net 86 "unconnected-(U3-RST-Pad15)")
+			(net 85 "unconnected-(U3-RST-Pad15)")
 			(pinfunction "RST")
 			(pintype "bidirectional+no_connect")
@@
 			(layers "*.Cu" "B.Mask")
 			(remove_unused_layers no)
-			(net 87 "unconnected-(U3-P0.02-LF-Pad19)")
+			(net 86 "unconnected-(U3-P0.02-LF-Pad19)")
 			(pinfunction "P0.02-LF")
 			(pintype "bidirectional")
@@
 			(layers "*.Cu" "B.Mask")
 			(remove_unused_layers no)
-			(net 83 "LED_PWR")
+			(net 87 "LED_PWR")
 			(pinfunction "P1.02-LF")
 			(pintype "bidirectional")
@@
 		)
 		(property ki_fp_filters "TO-???* *_Diode_* *SingleDiode* D_*")
-		(sheetname "/left/")
+		(sheetname "/right/")
 		(sheetfile "half.kicad_sch")
 		(attr smd)
@@
 		)
 		(property ki_fp_filters "TO-???* *_Diode_* *SingleDiode* D_*")
-		(sheetname "/left/")
+		(sheetname "/right/")
 		(sheetfile "half.kicad_sch")
 		(attr smd)
@@
 		)
 		(property ki_fp_filters "TO-???* *_Diode_* *SingleDiode* D_*")
-		(sheetname "/left/")
+		(sheetname "/right/")
 		(sheetfile "half.kicad_sch")
 		(attr smd)
@@
 		)
 		(property ki_fp_filters "TO-???* *_Diode_* *SingleDiode* D_*")
-		(sheetname "/left/")
+		(sheetname "/right/")
 		(sheetfile "half.kicad_sch")
 		(attr smd)
@@
 		)
 		(property ki_fp_filters "TO-???* *_Diode_* *SingleDiode* D_*")
-		(sheetname "/left/")
+		(sheetname "/right/")
 		(sheetfile "half.kicad_sch")
 		(attr smd)
@@
 		)
 		(property ki_fp_filters "TO-???* *_Diode_* *SingleDiode* D_*")
-		(sheetname "/left/")
+		(sheetname "/right/")
 		(sheetfile "half.kicad_sch")
 		(attr smd)
@@
 		)
 		(property ki_fp_filters "TO-???* *_Diode_* *SingleDiode* D_*")
-		(sheetname "/left/")
+		(sheetname "/right/")
 		(sheetfile "half.kicad_sch")
 		(attr smd)
@@
 		)
 		(property ki_fp_filters "TO-???* *_Diode_* *SingleDiode* D_*")
-		(sheetname "/left/")
+		(sheetname "/right/")
 		(sheetfile "half.kicad_sch")
 		(attr smd)
@@
 		)
 		(property ki_fp_filters "TO-???* *_Diode_* *SingleDiode* D_*")
-		(sheetname "/left/")
+		(sheetname "/right/")
 		(sheetfile "half.kicad_sch")
 		(attr smd)
@@
 		)
 		(property ki_fp_filters "TO-???* *_Diode_* *SingleDiode* D_*")
-		(sheetname "/left/")
+		(sheetname "/right/")
 		(sheetfile "half.kicad_sch")
 		(attr smd)
@@
 		)
 		(property ki_fp_filters "TO-???* *_Diode_* *SingleDiode* D_*")
-		(sheetname "/left/")
+		(sheetname "/right/")
 		(sheetfile "half.kicad_sch")
 		(attr smd)
@@
 		)
 		(property ki_fp_filters "TO-???* *_Diode_* *SingleDiode* D_*")
-		(sheetname "/left/")
+		(sheetname "/right/")
 		(sheetfile "half.kicad_sch")
 		(attr smd)
@@
 	)
 	(gr_poly
+		(pts
+			(xy 266 166) (xy 324 160) (xy 345 160) (xy 404 168) (xy 404 247) (xy 407 258) (xy 396 277) (xy 381 272)
+			(xy 351 266) (xy 300 266) (xy 264 246) (xy 264 170)
+		)
+		(stroke
+			(width 0.05)
+			(type solid)
+		)
+		(fill no)
+		(layer "Edge.Cuts")
+	)
+	(gr_poly

Commit message: placed components
Parts:
- removed D100, D103, D104, D107, D108, D111, D112, D115, D61, D63, D65, D67, D69, D71, D73, D75, D77, D79, D81, D83, D85, D87, D89, D91, D93, D95, D97, D99: SK6812MINI, LED_SMD:LED_SK6812MINI_PLCC4_3.5x3.5mm_P1.75mm
- added D10: D, Diode_SMD:D_SOD-123, B.Cu at (123.9, 122.2)
- added D11: D, Diode_SMD:D_SOD-123, B.Cu at (142.9, 125.0)
- added D12: D, Diode_SMD:D_SOD-123, B.Cu at (162.0, 127.9)
- added D19: D, Diode_SMD:D_SOD-123, B.Cu at (66.8, 166.0)
- added D2: D, Diode_SMD:D_SOD-123, B.Cu at (85.8, 108.8)
- added D20: D, Diode_SMD:D_SOD-123, B.Cu at (85.8, 166.0)
- added D21: D, Diode_SMD:D_SOD-123, B.Cu at (104.8, 163.1)
- added D22: D, Diode_SMD:D_SOD-123, B.Cu at (123.9, 160.2)
- added D23: D, Diode_SMD:D_SOD-123, B.Cu at (142.9, 163.1)
- added D24: D, Diode_SMD:D_SOD-123, B.Cu at (162.0, 166.0)
- added D31: D, Diode_SMD:D_SOD-123, B.Cu at (257.2, 104.1)
- added D32: D, Diode_SMD:D_SOD-123, B.Cu at (276.3, 103.1)
- added D33: D, Diode_SMD:D_SOD-123, B.Cu at (295.4, 106.0)
- added D34: D, Diode_SMD:D_SOD-123, B.Cu at (314.4, 108.8)
- added D35: D, Diode_SMD:D_SOD-123, B.Cu at (333.4, 108.8)
- added D36: D, Diode_SMD:D_SOD-123, B.Cu at (238.2, 127.9)
- added D4: D, Diode_SMD:D_SOD-123, B.Cu at (123.9, 103.1)
- added D43: D, Diode_SMD:D_SOD-123, B.Cu at (257.2, 144.1)
- added D44: D, Diode_SMD:D_SOD-123, B.Cu at (276.3, 141.2)
- added D45: D, Diode_SMD:D_SOD-123, B.Cu at (295.4, 144.1)
- added D46: D, Diode_SMD:D_SOD-123, B.Cu at (314.4, 146.9)
- added D47: D, Diode_SMD:D_SOD-123, B.Cu at (333.4, 146.9)
- added D48: D, Diode_SMD:D_SOD-123, B.Cu at (238.2, 166.0)
- added D55: D, Diode_SMD:D_SOD-123, B.Cu at (241.2, 188.6)
- added D56: D, Diode_SMD:D_SOD-123, B.Cu at (262.0, 182.2)
- added D57: D, Diode_SMD:D_SOD-123, B.Cu at (281.1, 182.2)
- added D58: D, Diode_SMD:D_SOD-123, B.Cu at (300.1, 185.0)
- added D6: D, Diode_SMD:D_SOD-123, B.Cu at (162.0, 108.8)
- added H2: MountingHole, MountingHole:MountingHole_2.1mm, F.Cu at (220.0, 179.0)
- added H4: MountingHole, MountingHole:MountingHole_2.1mm, F.Cu at (323.0, 180.0)
- added H6: MountingHole, MountingHole:MountingHole_2.1mm, F.Cu at (253.0, 96.0)
- added H8: MountingHole, MountingHole:MountingHole_2.1mm, F.Cu at (316.0, 96.0)
- added J2: Conn_01x04_Pin, OLED-SSD1306:SSD1306-0.91-OLED-4pin-128x32, F.Cu at (230.0, 100.0)
- added J4: JST_PH, Connector_JST:JST_PH_S2B-PH-K_1x02_P2.00mm_Horizontal, F.Cu at (223.0, 148.0)
- added L1: SK6812MINI, marbastlib-choc:LED_choc_6028R-ROT, B.Cu at (75.1, 103.8)
- added L10: SK6812MINI, marbastlib-choc:LED_choc_6028R-ROT, B.Cu at (132.2, 117.2)
- added L11: SK6812MINI, marbastlib-choc:LED_choc_6028R-ROT, B.Cu at (151.3, 120.0)
- added L12: SK6812MINI, marbastlib-choc:LED_choc_6028R-ROT, B.Cu at (170.3, 122.9)
- added L13: SK6812MINI, marbastlib-choc:LED_choc_6028R-ROT, B.Cu at (75.1, 141.9)
- added L14: SK6812MINI, marbastlib-choc:LED_choc_6028R-ROT, B.Cu at (94.2, 141.9)
- added L15: SK6812MINI, marbastlib-choc:LED_choc_6028R-ROT, B.Cu at (113.2, 139.1)
- added L16: SK6812MINI, marbastlib-choc:LED_choc_6028R-ROT, B.Cu at (132.2, 136.2)
- added L17: SK6812MINI, marbastlib-choc:LED_choc_6028R-ROT, B.Cu at (151.3, 139.1)
- added L18: SK6812MINI, marbastlib-choc:LED_choc_6028R-ROT, B.Cu at (170.3, 141.9)
- added L19: SK6812MINI, marbastlib-choc:LED_choc_6028R-ROT, B.Cu at (75.1, 161.0)
- added L2: SK6812MINI, marbastlib-choc:LED_choc_6028R-ROT, B.Cu at (94.2, 103.8)
- added L20: SK6812MINI, marbastlib-choc:LED_choc_6028R-ROT, B.Cu at (94.2, 161.0)
- added L21: SK6812MINI, marbastlib-choc:LED_choc_6028R-ROT, B.Cu at (113.2, 158.1)
- added L22: SK6812MINI, marbastlib-choc:LED_choc_6028R-ROT, B.Cu at (132.2, 155.2)
- added L23: SK6812MINI, marbastlib-choc:LED_choc_6028R-ROT, B.Cu at (151.3, 158.1)
- added L24: SK6812MINI, marbastlib-choc:LED_choc_6028R-ROT, B.Cu at (170.3, 161.0)
- added L25: SK6812MINI, marbastlib-choc:LED_choc_6028R-ROT, B.Cu at (108.4, 180.0)
- added L26: SK6812MINI, marbastlib-choc:LED_choc_6028R-ROT, B.Cu at (127.5, 177.2)
- added L27: SK6812MINI, marbastlib-choc:LED_choc_6028R-ROT, B.Cu at (146.5, 177.2)
- added L28: SK6812MINI, marbastlib-choc:LED_choc_6028R-ROT, B.Cu at (168.5, 182.3)
- added L29: SK6812MINI, marbastlib-choc:LED_choc_6028R-ROT, B.Cu at (191.3, 186.3)
- added L3: SK6812MINI, marbastlib-choc:LED_choc_6028R-ROT, B.Cu at (113.2, 101.0)
- added L30: SK6812MINI, marbastlib-choc:LED_choc_6028R-ROT, B.Cu at (246.6, 103.8)
- added L31: SK6812MINI, marbastlib-choc:LED_choc_6028R-ROT, B.Cu at (265.6, 99.1)
- added L32: SK6812MINI, marbastlib-choc:LED_choc_6028R-ROT, B.Cu at (284.6, 98.1)
- added L33: SK6812MINI, marbastlib-choc:LED_choc_6028R-ROT, B.Cu at (303.7, 101.0)
- added L34: SK6812MINI, marbastlib-choc:LED_choc_6028R-ROT, B.Cu at (322.8, 103.8)
- added L35: SK6812MINI, marbastlib-choc:LED_choc_6028R-ROT, B.Cu at (341.8, 103.8)
- added L36: SK6812MINI, marbastlib-choc:LED_choc_6028R-ROT, B.Cu at (246.6, 122.9)
- added L37: SK6812MINI, marbastlib-choc:LED_choc_6028R-ROT, B.Cu at (265.6, 118.1)
- added L38: SK6812MINI, marbastlib-choc:LED_choc_6028R-ROT, B.Cu at (284.6, 117.2)
- added L39: SK6812MINI, marbastlib-choc:LED_choc_6028R-ROT, B.Cu at (303.7, 120.0)
- added L4: SK6812MINI, marbastlib-choc:LED_choc_6028R-ROT, B.Cu at (132.2, 98.1)
- added L40: SK6812MINI, marbastlib-choc:LED_choc_6028R-ROT, B.Cu at (322.8, 122.9)
- added L41: SK6812MINI, marbastlib-choc:LED_choc_6028R-ROT, B.Cu at (341.8, 122.9)
- added L42: SK6812MINI, marbastlib-choc:LED_choc_6028R-ROT, B.Cu at (246.6, 141.9)
- added L43: SK6812MINI, marbastlib-choc:LED_choc_6028R-ROT, B.Cu at (265.6, 139.1)
- added L44: SK6812MINI, marbastlib-choc:LED_choc_6028R-ROT, B.Cu at (284.6, 136.2)
- added L45: SK6812MINI, marbastlib-choc:LED_choc_6028R-ROT, B.Cu at (303.7, 139.1)
- added L46: SK6812MINI, marbastlib-choc:LED_choc_6028R-ROT, B.Cu at (322.8, 141.9)
- added L47: SK6812MINI, marbastlib-choc:LED_choc_6028R-ROT, B.Cu at (341.8, 141.9)
- added L48: SK6812MINI, marbastlib-choc:LED_choc_6028R-ROT, B.Cu at (246.6, 161.0)
- added L49: SK6812MINI, marbastlib-choc:LED_choc_6028R-ROT, B.Cu at (265.6, 158.1)
- added L5: SK6812MINI, marbastlib-choc:LED_choc_6028R-ROT, B.Cu at (151.3, 101.0)
- added L50: SK6812MINI, marbastlib-choc:LED_choc_6028R-ROT, B.Cu at (284.6, 155.2)
- added L51: SK6812MINI, marbastlib-choc:LED_choc_6028R-ROT, B.Cu at (303.7, 158.1)
- added L52: SK6812MINI, marbastlib-choc:LED_choc_6028R-ROT, B.Cu at (322.8, 161.0)
- added L53: SK6812MINI, marbastlib-choc:LED_choc_6028R-ROT, B.Cu at (341.8, 161.0)
- added L54: SK6812MINI, marbastlib-choc:LED_choc_6028R-ROT, B.Cu at (224.6, 186.8)
- added L55: SK6812MINI, marbastlib-choc:LED_choc_6028R-ROT, B.Cu at (248.0, 181.7)
- added L56: SK6812MINI, marbastlib-choc:LED_choc_6028R-ROT, B.Cu at (270.4, 177.2)
- added L57: SK6812MINI, marbastlib-choc:LED_choc_6028R-ROT, B.Cu at (289.4, 177.2)
- added L58: SK6812MINI, marbastlib-choc:LED_choc_6028R-ROT, B.Cu at (308.5, 180.0)
- added L6: SK6812MINI, marbastlib-choc:LED_choc_6028R-ROT, B.Cu at (170.3, 103.8)
- added L7: SK6812MINI, marbastlib-choc:LED_choc_6028R-ROT, B.Cu at (75.1, 122.9)
- added L8: SK6812MINI, marbastlib-choc:LED_choc_6028R-ROT, B.Cu at (94.2, 122.9)
- added L9: SK6812MINI, marbastlib-choc:LED_choc_6028R-ROT, B.Cu at (113.2, 120.0)
- added SW30: SW_Push, marbastlib-choc:SW_choc_v1_HS_CPG135001S30_1u, F.Cu at (246.6, 108.8)
- added SW31: SW_Push, marbastlib-choc:SW_choc_v1_HS_CPG135001S30_1u, F.Cu at (265.6, 104.1)
- added SW32: SW_Push, marbastlib-choc:SW_choc_v1_HS_CPG135001S30_1u, F.Cu at (284.6, 103.1)
- added SW33: SW_Push, marbastlib-choc:SW_choc_v1_HS_CPG135001S30_1u, F.Cu at (303.7, 106.0)
- added SW34: SW_Push, marbastlib-choc:SW_choc_v1_HS_CPG135001S30_1u, F.Cu at (322.8, 108.8)
- added SW35: SW_Push, marbastlib-choc:SW_choc_v1_HS_CPG135001S30_1u, F.Cu at (341.8, 108.8)
- added SW36: SW_Push, marbastlib-choc:SW_choc_v1_HS_CPG135001S30_1u, F.Cu at (246.6, 127.9)
- added SW37: SW_Push, marbastlib-choc:SW_choc_v1_HS_CPG135001S30_1u, F.Cu at (265.6, 123.1)
- added SW38: SW_Push, marbastlib-choc:SW_choc_v1_HS_CPG135001S30_1u, F.Cu at (284.6, 122.2)
- added SW39: SW_Push, marbastlib-choc:SW_choc_v1_HS_CPG135001S30_1u, F.Cu at (303.7, 125.0)
- added SW40: SW_Push, marbastlib-choc:SW_choc_v1_HS_CPG135001S30_1u, F.Cu at (322.8, 127.9)
- added SW41: SW_Push, marbastlib-choc:SW_choc_v1_HS_CPG135001S30_1u, F.Cu at (341.8, 127.9)
- added SW42: SW_Push, marbastlib-choc:SW_choc_v1_HS_CPG135001S30_1u, F.Cu at (246.6, 146.9)
- added SW43: SW_Push, marbastlib-choc:SW_choc_v1_HS_CPG135001S30_1u, F.Cu at (265.6, 144.1)
- added SW44: SW_Push, marbastlib-choc:SW_choc_v1_HS_CPG135001S30_1u, F.Cu at (284.6, 141.2)
- added SW45: SW_Push, marbastlib-choc:SW_choc_v1_HS_CPG135001S30_1u, F.Cu at (303.7, 144.1)
- added SW46: SW_Push, marbastlib-choc:SW_choc_v1_HS_CPG135001S30_1u, F.Cu at (322.8, 146.9)
- added SW47: SW_Push, marbastlib-choc:SW_choc_v1_HS_CPG135001S30_1u, F.Cu at (341.8, 146.9)
- added SW48: SW_Push, marbastlib-choc:SW_choc_v1_HS_CPG135001S30_1u, F.Cu at (246.6, 166.0)
- added SW49: SW_Push, marbastlib-choc:SW_choc_v1_HS_CPG135001S30_1u, F.Cu at (265.6, 163.1)
- added SW50: SW_Push, marbastlib-choc:SW_choc_v1_HS_CPG135001S30_1u, F.Cu at (284.6, 160.2)
- added SW51: SW_Push, marbastlib-choc:SW_choc_v1_HS_CPG135001S30_1u, F.Cu at (303.7, 163.1)
- added SW52: SW_Push, marbastlib-choc:SW_choc_v1_HS_CPG135001S30_1u, F.Cu at (322.8, 166.0)
- added SW53: SW_Push, marbastlib-choc:SW_choc_v1_HS_CPG135001S30_1u, F.Cu at (341.8, 166.0)
- added SW54: SW_Push, marbastlib-choc:SW_choc_v1_HS_CPG135001S30_1u, F.Cu at (227.1, 191.2)
- added SW55: SW_Push, marbastlib-choc:SW_choc_v1_HS_CPG135001S30_1u, F.Cu at (249.3, 186.5)
- added SW56: SW_Push, marbastlib-choc:SW_choc_v1_HS_CPG135001S30_1u, F.Cu at (270.4, 182.2)
- added SW57: SW_Push, marbastlib-choc:SW_choc_v1_HS_CPG135001S30_1u, F.Cu at (289.4, 182.2)
- added SW58: SW_Push, marbastlib-choc:SW_choc_v1_HS_CPG135001S30_1u, F.Cu at (308.5, 185.0)
- added SW60: RotaryEncoder_Switch, marbastlib-various:ROT_Alps_EC11E-Switch, F.Cu at (226.0, 161.0)
- added SW62: SW_SPDT, Button_Switch_SMD:SW_SPDT_PCM12, F.Cu at (216.0, 147.0)
- added U4: SuperMini nRF52840, marbastlib-xp-promicroish:SuperMini_nRF52840_AH_USBup, F.Cu at (224.0, 115.9)
- D54: value SK6812MINI -> D; footprint LED_SMD:LED_SK6812MINI_PLCC4_3.5x3.5mm_P1.75mm -> Diode_SMD:D_SOD-123; moved to B.Cu
- SW59: footprint Rotary_Encoder:RotaryEncoder_Alps_EC11E-Switch_Vertical_H20mm_MountingHoles -> marbastlib-various:ROT_Alps_EC11E-Switch
- moved D40 229.8 mm to (314.4, 127.9)
- moved D41 229.4 mm to (333.4, 127.9)
- moved D39 229.1 mm to (295.4, 125.0)
- moved D37 228.6 mm to (257.2, 123.1)
- moved D38 228.5 mm to (276.3, 122.2)
- moved D51 199.5 mm to (295.4, 163.1)
- moved D50 198.9 mm to (276.3, 160.2)
- moved D49 198.9 mm to (257.2, 163.1)
- moved D52 197.7 mm to (314.4, 166.0), turned to -90 degrees
- moved D53 194.0 mm to (333.4, 166.0), turned to -90 degrees
- moved D54 178.9 mm to (219.9, 195.3), turned to -60 degrees
- moved H3 143.4 mm to (196.0, 179.0), turned to 0 degrees
- moved D29 131.4 mm to (181.6, 186.4), turned to -120 degrees
- moved D28 130.5 mm to (159.1, 185.0), turned to -105 degrees
- moved D27 124.8 mm to (138.2, 182.2)
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Connections:
- D13 pad 1: ROW2 -> ROW3
- D14 pad 1: ROW2 -> ROW3
- D15 pad 1: ROW2 -> ROW3
- D16 pad 1: ROW2 -> ROW3
- D17 pad 1: ROW2 -> ROW3
- D18 pad 1: ROW2 -> ROW3
- D25 pad 1: ROW3 -> ROW5
- D26 pad 1: ROW3 -> ROW5
- D27 pad 1: ROW3 -> ROW5
- D28 pad 1: ROW3 -> ROW5
- D29 pad 1: ROW3 -> ROW5
- D30 pad 1: ROW3 -> ROW1
- D37 pad 1: ROW4 -> ROW2
- D38 pad 1: ROW4 -> ROW2
- D39 pad 1: ROW4 -> ROW2
- D40 pad 1: ROW4 -> ROW2
- D41 pad 1: ROW4 -> ROW2
- D42 pad 1: ROW4 -> ROW3
- D49 pad 1: ROW5 -> ROW4
- D50 pad 1: ROW5 -> ROW4
- D51 pad 1: ROW5 -> ROW4
- D52 pad 1: ROW5 -> ROW4
- D53 pad 1: ROW5 -> ROW4
- D54 pad 1: Net-(D54-DOUT) -> ROW5
- D54 pad 2: GND -> Net-(D54-A)
- D7 pad 1: ROW1 -> ROW2
- D8 pad 1: ROW1 -> ROW2
- D9 pad 1: ROW1 -> ROW2
- J1 pad 2: +3.3V -> VBAT
- SW10 pad 2: Net-(D16-A) -> Net-(D10-A)
- SW11 pad 2: Net-(D17-A) -> Net-(D11-A)
- SW12 pad 2: Net-(D18-A) -> Net-(D12-A)
- SW13 pad 2: Net-(D25-A) -> Net-(D13-A)
- SW14 pad 2: Net-(D26-A) -> Net-(D14-A)
- SW15 pad 2: Net-(D27-A) -> Net-(D15-A)
- SW16 pad 2: Net-(D28-A) -> Net-(D16-A)
- SW17 pad 2: Net-(D29-A) -> Net-(D17-A)
- SW18 pad 2: Net-(D30-A) -> Net-(D18-A)
- SW19 pad 2: Net-(D37-A) -> Net-(D19-A)
- SW2 pad 2: Net-(D3-A) -> Net-(D2-A)
- SW20 pad 2: Net-(D38-A) -> Net-(D20-A)
- SW21 pad 2: Net-(D39-A) -> Net-(D21-A)
- SW22 pad 2: Net-(D40-A) -> Net-(D22-A)
- SW23 pad 2: Net-(D41-A) -> Net-(D23-A)
- SW24 pad 2: Net-(D42-A) -> Net-(D24-A)
- SW25 pad 2: Net-(D49-A) -> Net-(D25-A)
- SW26 pad 2: Net-(D50-A) -> Net-(D26-A)
- SW27 pad 2: Net-(D51-A) -> Net-(D27-A)
- SW28 pad 2: Net-(D52-A) -> Net-(D28-A)
- SW29 pad 2: Net-(D53-A) -> Net-(D29-A)
- SW3 pad 2: Net-(D5-A) -> Net-(D3-A)
- SW4 pad 2: Net-(D7-A) -> Net-(D4-A)
- SW5 pad 2: Net-(D8-A) -> Net-(D5-A)
- SW6 pad 2: Net-(D9-A) -> Net-(D6-A)
- SW7 pad 2: Net-(D13-A) -> Net-(D7-A)
- SW8 pad 2: Net-(D14-A) -> Net-(D8-A)
- SW9 pad 2: Net-(D15-A) -> Net-(D9-A)
- U3 pad 26: LED_PWR -> unconnected-(U3-P1.02-LF-Pad26)
Routing:
- net Net-(J3-Pin_1): track 10.8 -> 0.00 mm
- net Net-(D37-A): track 10.1 -> 0.00 mm
- net Net-(D49-A): track 10.1 -> 0.00 mm
- net Net-(D25-A): track 10.1 -> 0.00 mm
- net Net-(D13-A): track 10.1 -> 0.00 mm
- net Net-(D1-A): track 10.1 -> 0.00 mm
- net Net-(D51-A): track 10.1 -> 0.00 mm
- net Net-(D50-A): track 10.1 -> 0.00 mm
- net Net-(D53-A): track 10.0 -> 0.00 mm
- net Net-(D52-A): track 9.57 -> 0.00 mm
Other:
- board size 380 x 251 mm -> 292 x 117 mm

Commit message: first route half
Parts:
- moved U4 2.33 mm to (225.0, 118.0)
- moved J1 2.24 mm to (197.0, 102.0)
- moved J2 2.24 mm to (231.0, 102.0)
- moved U3 2.24 mm to (191.0, 118.0)
- moved SW61 1.33 mm to (198.7, 147.0)
- moved SW62 1.00 mm to (217.0, 147.0)
Connections:
- U3 pad 13: unconnected-(U3-BAT+-Pad13) -> VBAT
- U3 pad 17: COL6 -> R_E_S
- U3 pad 18: COL5 -> COL6
- U3 pad 19: unconnected-(U3-P0.02-LF-Pad19) -> COL5
- U3 pad 24: R_E_S -> ROW5
- U3 pad 25: ROW5 -> unconnected-(U3-P1.01-LF-Pad25)
- U4 pad 13: unconnected-(U4-BAT+-Pad13) -> VBAT
- U4 pad 17: COL6 -> R_E_S
- U4 pad 18: COL5 -> COL6
- U4 pad 19: unconnected-(U4-P0.02-LF-Pad19) -> COL5
- U4 pad 24: R_E_S -> ROW5
- U4 pad 25: ROW5 -> unconnected-(U4-P1.01-LF-Pad25)
Routing:
- net +3.3V: track 0.00 -> 748.5 mm
- net COL1: track 0.00 -> 279.8 mm, vias 0 -> 3
- net COL2: track 0.00 -> 225.1 mm, vias 0 -> 5
- net COL3: track 0.00 -> 177.4 mm, vias 0 -> 7
- net COL4: track 0.00 -> 170.2 mm, vias 0 -> 5
- net ROW5: track 0.00 -> 154.9 mm, vias 0 -> 4
- net COL5: track 0.00 -> 154.3 mm, vias 0 -> 1
- net ROW4: track 0.00 -> 152.1 mm
- net LED_DAT: track 0.00 -> 144.2 mm, vias 0 -> 1
- net ROW1: track 0.00 -> 134.6 mm, vias 0 -> 2
- net ROW3: track 0.00 -> 129.6 mm, vias 0 -> 2
- net ROW2: track 0.00 -> 123.2 mm
- net Net-(L6-DOUT): track 0.00 -> 104.8 mm, vias 0 -> 4
- net Net-(L18-DOUT): track 0.00 -> 103.9 mm, vias 0 -> 4
- net Net-(L12-DOUT): track 0.00 -> 103.8 mm, vias 0 -> 4
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- added copper zone on B.Cu, net GND
- added copper zone on F.Cu, net GND
Other:
- board size 292 x 117 mm -> 292.1 x 116.2 mm
