File: PCB/keeby.kicad_pcb (KiCad board)
At the start: 2 copper layers, 292.1 x 116.2 mm, 192 parts, among them J1 Conn_01x04_Pin, J2 Conn_01x04_Pin, J3 JST_PH, J4 JST_PH, SW1 SW_Push, SW10 SW_Push, SW11 SW_Push, SW12 SW_Push, SW13 SW_Push, SW14 SW_Push, SW15 SW_Push, SW16 SW_Push, SW17 SW_Push, SW18 SW_Push, SW19 SW_Push, SW2 SW_Push, SW20 SW_Push, SW21 SW_Push, SW22 SW_Push, SW23 SW_Push, SW24 SW_Push, SW25 SW_Push, SW26 SW_Push, SW27 SW_Push, SW28 SW_Push, SW29 SW_Push, SW3 SW_Push, SW30 SW_Push, SW31 SW_Push, SW32 SW_Push, SW33 SW_Push, SW34 SW_Push, SW35 SW_Push, SW36 SW_Push, SW37 SW_Push, SW38 SW_Push, SW39 SW_Push, SW4 SW_Push, SW40 SW_Push, SW41 SW_Push, SW42 SW_Push, SW43 SW_Push, SW44 SW_Push, SW45 SW_Push, SW46 SW_Push, SW47 SW_Push, SW48 SW_Push, SW49 SW_Push, SW5 SW_Push, SW50 SW_Push, SW51 SW_Push, SW52 SW_Push, SW53 SW_Push, SW54 SW_Push, SW55 SW_Push, SW56 SW_Push, SW57 SW_Push, SW58 SW_Push, SW59 RotaryEncoder_Switch, SW6 SW_Push, SW60 RotaryEncoder_Switch, SW61 SW_SPDT, SW62 SW_SPDT, SW7 SW_Push, SW8 SW_Push, SW9 SW_Push, U3 SuperMini nRF52840, U4 SuperMini nRF52840

Commit message: flipped the switches to be on the right side
Parts:
- J3, J4, SW1, SW10, SW11, SW12, SW13, SW14, SW15, SW16, SW17, SW18, SW19, SW2, SW20, SW21, SW22, SW23, SW24, SW25, SW26, SW27, SW28, SW29, SW3, SW30, SW31, SW32, SW33, SW34, SW35, SW36, SW37, SW38, SW39, SW4, SW40, SW41, SW42, SW43, SW44, SW45, SW46, SW47, SW48, SW49, SW5, SW50, SW51, SW52, SW53, SW54, SW55, SW56, SW57, SW58, SW6, SW7, SW8, SW9: moved to B.Cu
- moved D11 16.8 mm to (158.9, 130.2)
- moved D13 16.8 mm to (82.8, 152.2)
- moved D14 16.8 mm to (101.8, 152.2)
- moved D16 16.8 mm to (139.9, 146.4)
- moved D18 16.8 mm to (178.0, 152.2)
- moved D21 16.8 mm to (120.8, 168.3)
- moved D22 16.8 mm to (139.9, 165.5)
- moved D23 16.8 mm to (158.9, 168.3)
- moved D25 16.8 mm to (116.1, 190.2)
- moved D27 16.8 mm to (154.2, 187.4)
- moved D39 16.8 mm to (311.4, 130.2)
- moved D42 16.8 mm to (254.2, 152.2)
- moved D44 16.8 mm to (292.3, 146.4)
- moved D46 16.8 mm to (330.4, 152.2)
- moved D47 16.8 mm to (349.4, 152.2)
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Routing:
- net +3.3V: track 1618.5 -> 0.00 mm, vias 39 -> 0
- net COL1: track 395.7 -> 0.00 mm, vias 4 -> 0
- net COL5: track 381.5 -> 0.00 mm, vias 10 -> 0
- net COL4: track 375.9 -> 0.00 mm, vias 13 -> 0
- net COL6: track 369.9 -> 0.00 mm, vias 8 -> 0
- net COL2: track 363.9 -> 0.00 mm, vias 8 -> 0
- net COL3: track 344.8 -> 0.00 mm, vias 14 -> 0
- net ROW5: track 330.4 -> 0.00 mm, vias 11 -> 0
- net ROW4: track 302.1 -> 0.00 mm, vias 2 -> 0
- net ROW1: track 276.1 -> 0.00 mm, vias 8 -> 0
- net ROW3: track 263.4 -> 0.00 mm, vias 3 -> 0
- net ROW2: track 245.7 -> 0.00 mm
- net LED_DAT: track 187.6 -> 0.00 mm, vias 3 -> 0
- net Net-(L53-DOUT): track 130.3 -> 0.00 mm, vias 4 -> 0
- net R_E_1: track 119.6 -> 0.00 mm, vias 5 -> 0
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
Commit message: fixing routing
Parts:
- SW61, SW62: moved to B.Cu
- moved D27 18.2 mm to (139.4, 176.8), turned to 90 degrees
- moved D56 18.2 mm to (263.2, 176.8), turned to 90 degrees
- moved D57 18.2 mm to (282.3, 176.8), turned to 90 degrees
- moved D25 18.2 mm to (101.3, 179.7), turned to 90 degrees
- moved D58 18.2 mm to (301.3, 179.7), turned to 90 degrees
- moved D26 18.2 mm to (120.3, 176.8), turned to 90 degrees
- moved D28 17.0 mm to (175.6, 189.0), turned to 75 degrees
- moved D29 17.0 mm to (196.4, 194.6), turned to 60 degrees
- moved D54 16.5 mm to (234.0, 186.8), turned to 120 degrees
- moved D55 16.5 mm to (257.0, 184.1), turned to 105 degrees
- moved L25 9.91 mm to (108.9, 189.9), turned to 0 degrees
- moved L26 9.91 mm to (128.0, 187.1), turned to 0 degrees
- moved L27 9.91 mm to (147.0, 187.1), turned to 0 degrees
- moved L56 9.91 mm to (270.9, 187.1), turned to 0 degrees
- moved L57 9.91 mm to (289.9, 187.1), turned to 0 degrees
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Routing:
- net COL4: track 0.00 -> 57.2 mm
- net COL2: track 0.00 -> 57.2 mm
- net COL1: track 0.00 -> 57.2 mm
- net COL3: track 0.00 -> 57.1 mm

Commit message: switch aligned with led
Parts:
- moved D27 18.2 mm to (154.2, 187.4), turned to -90 degrees
- moved D25 18.2 mm to (116.1, 190.2), turned to -90 degrees
- moved D26 18.2 mm to (135.1, 187.4), turned to -90 degrees
- moved D28 17.0 mm to (159.1, 185.0), turned to -105 degrees
- moved D29 17.0 mm to (181.6, 186.4), turned to -120 degrees
- moved L25 9.91 mm to (108.4, 180.0), turned to 180 degrees
- moved L26 9.91 mm to (127.5, 177.2), turned to 180 degrees
- moved L27 9.91 mm to (146.5, 177.2), turned to 180 degrees
- moved L28 9.65 mm to (168.5, 182.3), turned to 165 degrees
- moved L29 9.65 mm to (191.3, 186.3), turned to 150 degrees
- moved D31 1.86 mm to (273.2, 111.2)
- moved L31 1.86 mm to (265.6, 100.9)
- moved L37 1.86 mm to (265.6, 120.0)
- moved D37 1.86 mm to (273.2, 130.2)
- moved SW31 1.55 mm to (265.6, 105.6)
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- renumbered SW5 to SW1, SW9 to SW10, SW10 to SW11, SW11 to SW12, SW18 to SW13, SW13 to SW14, SW14 to SW15, SW15 to SW16, SW16 to SW17, SW17 to SW18, SW24 to SW19, SW1 to SW2, SW19 to SW20, SW20 to SW21, SW21 to SW22, SW22 to SW23, SW23 to SW24, SW2 to SW3, SW3 to SW4, SW4 to SW5, SW12 to SW7, SW7 to SW8, SW8 to SW9
Routing:
- net COL4: track 57.2 -> 0.00 mm
- net COL2: track 57.2 -> 0.00 mm
- net COL1: track 57.2 -> 0.00 mm
- net COL3: track 57.1 -> 0.00 mm

Commit message: prepare complete redesign
Parts:
- S61: renamed from SW61; value SW_SPDT -> S_SPDT
- S62: renamed from SW62; value SW_SPDT -> S_SPDT
- moved D12 164.2 mm to (32.1, 57.9), turned to 90 degrees
- moved D18 164.2 mm to (32.1, 76.9), turned to 90 degrees
- moved D24 164.2 mm to (32.1, 96.0), turned to 90 degrees
- moved D6 164.2 mm to (32.1, 38.8), turned to 90 degrees
- moved SW1 147.2 mm to (38.1, 43.8), turned to 0 degrees
- moved SW13 147.2 mm to (38.1, 81.9), turned to 0 degrees
- moved SW19 147.2 mm to (38.1, 101.0), turned to 0 degrees
- moved SW7 147.2 mm to (38.1, 62.9), turned to 0 degrees
- moved D31 92.2 mm to (222.6, 34.1), turned to 90 degrees
- moved D37 92.2 mm to (222.6, 53.1), turned to 90 degrees
- moved D39 90.7 mm to (260.7, 55.0), turned to 90 degrees
- moved D51 90.7 mm to (260.7, 93.1), turned to 90 degrees
- moved D27 90.7 mm to (103.5, 112.2), turned to 90 degrees
- moved D33 90.7 mm to (260.7, 36.0), turned to 90 degrees
- moved D38 90.7 mm to (241.7, 52.1), turned to 90 degrees
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- renumbered SW59 to S59, SW60 to S60, SW6 to SW1, SW1 to SW6
