File: PCB/keeby.kicad_pcb (KiCad board)
At the start: 2 copper layers, 292.1 x 116.2 mm, 192 parts, among them J1 Conn_01x04_Pin, J2 Conn_01x04_Pin, J3 JST_PH, J4 JST_PH, SW1 SW_Push, SW10 SW_Push, SW11 SW_Push, SW12 SW_Push, SW13 SW_Push, SW14 SW_Push, SW15 SW_Push, SW16 SW_Push, SW17 SW_Push, SW18 SW_Push, SW19 SW_Push, SW2 SW_Push, SW20 SW_Push, SW21 SW_Push, SW22 SW_Push, SW23 SW_Push, SW24 SW_Push, SW25 SW_Push, SW26 SW_Push, SW27 SW_Push, SW28 SW_Push, SW29 SW_Push, SW3 SW_Push, SW30 SW_Push, SW31 SW_Push, SW32 SW_Push, SW33 SW_Push, SW34 SW_Push, SW35 SW_Push, SW36 SW_Push, SW37 SW_Push, SW38 SW_Push, SW39 SW_Push, SW4 SW_Push, SW40 SW_Push, SW41 SW_Push, SW42 SW_Push, SW43 SW_Push, SW44 SW_Push, SW45 SW_Push, SW46 SW_Push, SW47 SW_Push, SW48 SW_Push, SW49 SW_Push, SW5 SW_Push, SW50 SW_Push, SW51 SW_Push, SW52 SW_Push, SW53 SW_Push, SW54 SW_Push, SW55 SW_Push, SW56 SW_Push, SW57 SW_Push, SW58 SW_Push, SW59 RotaryEncoder_Switch, SW6 SW_Push, SW60 RotaryEncoder_Switch, SW61 SW_SPDT, SW62 SW_SPDT, SW7 SW_Push, SW8 SW_Push, SW9 SW_Push, U3 SuperMini nRF52840, U4 SuperMini nRF52840

Commit message: prepared outline
Parts:
- removed H1, H2, H3, H4, H5, H6, H7, H8: MountingHole, MountingHole:MountingHole_2.1mm
- J3, J4, SW25, SW26, SW27, SW28, SW29, SW30, SW31, SW32, SW33, SW34, SW35, SW36, SW37, SW38, SW39, SW40, SW41, SW42, SW43, SW44, SW45, SW46, SW47, SW48, SW49, SW50, SW51, SW52, SW53, SW54, SW55, SW56, SW57, SW58: moved to B.Cu
- S61: renamed from SW61; value SW_SPDT -> S_SPDT; moved to B.Cu
- S62: renamed from SW62; value SW_SPDT -> S_SPDT; moved to B.Cu
- SW1: renamed from SW6; moved to B.Cu
- SW10: renamed from SW9; moved to B.Cu
- SW11: renamed from SW10; moved to B.Cu
- SW12: renamed from SW11; moved to B.Cu
- SW13: renamed from SW18; moved to B.Cu
- SW14: renamed from SW13; moved to B.Cu
- SW15: renamed from SW14; moved to B.Cu
- SW16: renamed from SW15; moved to B.Cu
- SW17: renamed from SW16; moved to B.Cu
- SW18: renamed from SW17; moved to B.Cu
- SW19: renamed from SW24; moved to B.Cu
- SW2: renamed from SW1; moved to B.Cu
- SW20: renamed from SW19; moved to B.Cu
- SW21: renamed from SW20; moved to B.Cu
- SW22: renamed from SW21; moved to B.Cu
- SW23: renamed from SW22; moved to B.Cu
- SW24: renamed from SW23; moved to B.Cu
- SW3: renamed from SW2; moved to B.Cu
- SW4: renamed from SW3; moved to B.Cu
- SW5: renamed from SW4; moved to B.Cu
- SW6: renamed from SW5; moved to B.Cu
- SW7: renamed from SW12; moved to B.Cu
- SW8: renamed from SW7; moved to B.Cu
- SW9: renamed from SW8; moved to B.Cu
- moved SW1 145.3 mm to (38.1, 48.6)
- moved SW13 145.3 mm to (38.1, 86.7)
- moved SW19 145.3 mm to (38.1, 105.7)
- moved SW7 145.3 mm to (38.1, 67.6)
- moved D12 144.9 mm to (32.4, 63.1), turned to 90 degrees
- moved D18 144.9 mm to (32.4, 82.2), turned to 90 degrees
- moved D24 144.9 mm to (32.4, 101.2), turned to 90 degrees
- moved D6 144.9 mm to (32.4, 44.1), turned to 90 degrees
- moved D26 77.5 mm to (84.7, 112.7), turned to 90 degrees
- moved D27 77.5 mm to (103.8, 112.7), turned to 90 degrees
- moved D25 77.5 mm to (65.7, 115.5), turned to 90 degrees
- moved SW26 74.8 mm to (90.5, 117.2)
- moved SW27 74.8 mm to (109.5, 117.2)
- moved SW25 74.8 mm to (71.4, 120.0)
- moved J1 74.2 mm to (163.0, 36.0)
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- renumbered SW59 to S59, SW60 to S60
Routing:
- net +3.3V: track 1618.5 -> 0.00 mm, vias 39 -> 0
- net COL1: track 395.7 -> 0.00 mm, vias 4 -> 0
- net COL5: track 381.5 -> 0.00 mm, vias 10 -> 0
- net COL4: track 375.9 -> 0.00 mm, vias 13 -> 0
- net COL6: track 369.9 -> 0.00 mm, vias 8 -> 0
- net COL2: track 363.9 -> 0.00 mm, vias 8 -> 0
- net COL3: track 344.8 -> 0.00 mm, vias 14 -> 0
- net ROW5: track 330.4 -> 0.00 mm, vias 11 -> 0
- net ROW4: track 302.1 -> 0.00 mm, vias 2 -> 0
- net ROW1: track 276.1 -> 0.00 mm, vias 8 -> 0
- net ROW3: track 263.4 -> 0.00 mm, vias 3 -> 0
- net ROW2: track 245.7 -> 0.00 mm
- net LED_DAT: track 187.6 -> 0.00 mm, vias 3 -> 0
- net Net-(L53-DOUT): track 130.3 -> 0.00 mm, vias 4 -> 0
- net R_E_1: track 119.6 -> 0.00 mm, vias 5 -> 0
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Other:
- board size 292.1 x 116.2 mm -> 147.6 x 127.8 mm

Commit message: started routing
Other:
- board size 147.6 x 127.8 mm -> 313.2 x 127.8 mm

Commit message: progress??
Routing:
- net Net-(D6-A): track 0.00 -> 2.59 mm
- net Net-(D35-A): track 0.00 -> 2.59 mm

Commit message: Revert "progress??"
This reverts commit cc348a77a973bafb10792190f59578297f7118eb.
Routing:
- net Net-(D6-A): track 2.59 -> 0.00 mm
- net Net-(D35-A): track 2.59 -> 0.00 mm

Commit message: fixing leds
Parts:
- added H1: MountingHole, MountingHole:MountingHole_2.1mm, F.Cu at (180.9, 23.9)
- added H2: MountingHole, MountingHole:MountingHole_2.1mm, F.Cu at (177.2, 102.8)
- added H3: MountingHole, MountingHole:MountingHole_2.1mm, F.Cu at (180.9, 29.7)
- added H4: MountingHole, MountingHole:MountingHole_2.1mm, F.Cu at (177.2, 108.5)
- added H5: MountingHole, MountingHole:MountingHole_2.1mm, F.Cu at (180.9, 35.5)
- added H6: MountingHole, MountingHole:MountingHole_2.1mm, F.Cu at (177.2, 114.2)
- added H7: MountingHole, MountingHole:MountingHole_2.1mm, F.Cu at (180.9, 41.2)
- added H8: MountingHole, MountingHole:MountingHole_2.1mm, F.Cu at (177.2, 120.0)
- L1, L10, L11, L12, L13, L14, L15, L16, L17, L18, L19, L2, L20, L21, L22, L23, L24, L25, L26, L27, L28, L29, L3, L30, L31, L32, L33, L34, L35, L36, L37, L38, L39, L4, L40, L41, L42, L43, L44, L45, L46, L47, L48, L49, L5, L50, L51, L52, L53, L54, L55, L56, L57, L58, L6, L7, L8, L9: value SK6812MINI -> SK6812-MINI-E
- U4: moved to B.Cu
- moved D55 3.00 mm to (222.5, 120.1), turned to -75 degrees
- moved D28 3.00 mm to (128.3, 117.1), turned to -105 degrees
- moved D1 3.00 mm to (51.4, 36.3), turned to -90 degrees
- moved D10 3.00 mm to (108.5, 52.5), turned to -90 degrees
- moved D11 3.00 mm to (127.6, 55.4), turned to -90 degrees
- moved D12 3.00 mm to (32.4, 60.1), turned to -90 degrees
- moved D13 3.00 mm to (51.4, 74.4), turned to -90 degrees
- moved D14 3.00 mm to (70.5, 71.6), turned to -90 degrees
- moved D15 3.00 mm to (89.5, 68.7), turned to -90 degrees
- moved D16 3.00 mm to (108.5, 71.6), turned to -90 degrees
- moved D17 3.00 mm to (127.6, 74.4), turned to -90 degrees
- moved D18 3.00 mm to (32.4, 79.2), turned to -90 degrees
- moved D19 3.00 mm to (51.4, 93.5), turned to -90 degrees
- moved D2 3.00 mm to (70.5, 33.5), turned to -90 degrees
- moved D20 3.00 mm to (70.5, 90.6), turned to -90 degrees
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Connections:
- D1 pad 1: ROW1 -> /left/ROW1
- D10 pad 1: ROW2 -> /left/ROW2
- D11 pad 1: ROW2 -> /left/ROW2
- D12 pad 1: ROW2 -> /left/ROW2
- D13 pad 1: ROW3 -> /left/ROW3
- D14 pad 1: ROW3 -> /left/ROW3
- D15 pad 1: ROW3 -> /left/ROW3
- D16 pad 1: ROW3 -> /left/ROW3
- D17 pad 1: ROW3 -> /left/ROW3
- D18 pad 1: ROW3 -> /left/ROW3
- D19 pad 1: ROW4 -> /left/ROW4
- D2 pad 1: ROW1 -> /left/ROW1
- D20 pad 1: ROW4 -> /left/ROW4
- D21 pad 1: ROW4 -> /left/ROW4
- D22 pad 1: ROW4 -> /left/ROW4
- D23 pad 1: ROW4 -> /left/ROW4
- D24 pad 1: ROW4 -> /left/ROW4
- D25 pad 1: ROW5 -> /left/ROW5
- D26 pad 1: ROW5 -> /left/ROW5
- D27 pad 1: ROW5 -> /left/ROW5
- D28 pad 1: ROW5 -> /left/ROW5
- D29 pad 1: ROW5 -> /left/ROW5
- D3 pad 1: ROW1 -> /left/ROW1
- D30 pad 1: ROW1 -> /right/ROW1
- D31 pad 1: ROW1 -> /right/ROW1
- D32 pad 1: ROW1 -> /right/ROW1
- D33 pad 1: ROW1 -> /right/ROW1
- D34 pad 1: ROW1 -> /right/ROW1
- D35 pad 1: ROW1 -> /right/ROW1
- D36 pad 1: ROW2 -> /right/ROW2
- D37 pad 1: ROW2 -> /right/ROW2
- D38 pad 1: ROW2 -> /right/ROW2
- D39 pad 1: ROW2 -> /right/ROW2
- D4 pad 1: ROW1 -> /left/ROW1
- D40 pad 1: ROW2 -> /right/ROW2
- D41 pad 1: ROW2 -> /right/ROW2
- D42 pad 1: ROW3 -> /right/ROW3
- D43 pad 1: ROW3 -> /right/ROW3
- D44 pad 1: ROW3 -> /right/ROW3
- D45 pad 1: ROW3 -> /right/ROW3
- D46 pad 1: ROW3 -> /right/ROW3
- D47 pad 1: ROW3 -> /right/ROW3
- D48 pad 1: ROW4 -> /right/ROW4
- D49 pad 1: ROW4 -> /right/ROW4
- D5 pad 1: ROW1 -> /left/ROW1
- D50 pad 1: ROW4 -> /right/ROW4
- D51 pad 1: ROW4 -> /right/ROW4
- D52 pad 1: ROW4 -> /right/ROW4
- D53 pad 1: ROW4 -> /right/ROW4
- D54 pad 1: ROW5 -> /right/ROW5
- D55 pad 1: ROW5 -> /right/ROW5
- D56 pad 1: ROW5 -> /right/ROW5
- D57 pad 1: ROW5 -> /right/ROW5
- D58 pad 1: ROW5 -> /right/ROW5
- D6 pad 1: ROW1 -> /left/ROW1
- D7 pad 1: ROW2 -> /left/ROW2
- D8 pad 1: ROW2 -> /left/ROW2
- D9 pad 1: ROW2 -> /left/ROW2
- J1 pad 2: VBAT -> /left/VBAT
- J1 pad 3: SCL -> /left/SCL
- J1 pad 4: SDA -> /left/SDA
- J2 pad 2: VBAT -> /right/VBAT
- J2 pad 3: SCL -> /right/SCL
- J2 pad 4: SDA -> /right/SDA
- L1 pad 3: LED_DAT -> Net-(L1-DIN)
- L13 pad 3: Net-(L12-DOUT) -> Net-(L13-DIN)
- L16 pad 1: +3.3V -> GND
- L16 pad 3: Net-(L15-DOUT) -> Net-(L16-DIN)
- L16 pad 4: GND -> +3.3V
- L17 pad 1: +3.3V -> GND
- L17 pad 4: GND -> +3.3V
- L18 pad 1: +3.3V -> GND
- L18 pad 4: GND -> +3.3V
- L19 pad 1: +3.3V -> GND
- L19 pad 4: GND -> +3.3V
- L20 pad 1: +3.3V -> GND
- L20 pad 2: Net-(L20-DOUT) -> unconnected-(L20-DOUT-Pad2)
- L20 pad 4: GND -> +3.3V
- L21 pad 1: +3.3V -> GND
- L21 pad 3: Net-(L20-DOUT) -> Net-(L16-DIN)
- L21 pad 4: GND -> +3.3V
- L22 pad 1: +3.3V -> GND
- L22 pad 4: GND -> +3.3V
- L23 pad 1: +3.3V -> GND
- L23 pad 4: GND -> +3.3V
- L24 pad 1: +3.3V -> GND
- L24 pad 4: GND -> +3.3V
- L25 pad 1: +3.3V -> GND
- L25 pad 4: GND -> +3.3V
- L26 pad 1: +3.3V -> GND
- L26 pad 2: Net-(L26-DOUT) -> Net-(L13-DIN)
- L26 pad 4: GND -> +3.3V
- L27 pad 1: +3.3V -> GND
- L27 pad 3: Net-(L26-DOUT) -> Net-(L12-DOUT)
- L27 pad 4: GND -> +3.3V
- L28 pad 1: +3.3V -> GND
- L28 pad 4: GND -> +3.3V
- L29 pad 1: +3.3V -> GND
- L29 pad 2: unconnected-(L29-DOUT-Pad2) -> Net-(L15-DOUT)
- L29 pad 4: GND -> +3.3V
- L30 pad 3: LED_DAT -> Net-(L30-DIN)
- L35 pad 2: Net-(L35-DOUT) -> /right/LED_DAT
- L36 pad 3: Net-(L35-DOUT) -> Net-(L30-DIN)
- L42 pad 3: Net-(L41-DOUT) -> Net-(L42-DIN)
- L45 pad 1: +3.3V -> GND
- L45 pad 3: Net-(L44-DOUT) -> Net-(L45-DIN)
- L45 pad 4: GND -> +3.3V
- L46 pad 1: +3.3V -> GND
- L46 pad 4: GND -> +3.3V
- L47 pad 1: +3.3V -> GND
- L47 pad 4: GND -> +3.3V
- L48 pad 1: +3.3V -> GND
- L48 pad 4: GND -> +3.3V
- L49 pad 1: +3.3V -> GND
- L49 pad 2: Net-(L49-DOUT) -> unconnected-(L49-DOUT-Pad2)
- L49 pad 4: GND -> +3.3V
- L50 pad 1: +3.3V -> GND
- L50 pad 3: Net-(L49-DOUT) -> Net-(L45-DIN)
- L50 pad 4: GND -> +3.3V
- L51 pad 1: +3.3V -> GND
- L51 pad 4: GND -> +3.3V
- L52 pad 1: +3.3V -> GND
- L52 pad 4: GND -> +3.3V
- L53 pad 1: +3.3V -> GND
- L53 pad 4: GND -> +3.3V
- L54 pad 1: +3.3V -> GND
- L54 pad 4: GND -> +3.3V
- L55 pad 1: +3.3V -> GND
- L55 pad 2: Net-(L55-DOUT) -> Net-(L42-DIN)
- L55 pad 4: GND -> +3.3V
- L56 pad 1: +3.3V -> GND
- L56 pad 3: Net-(L55-DOUT) -> Net-(L41-DOUT)
- L56 pad 4: GND -> +3.3V
- L57 pad 1: +3.3V -> GND
- L57 pad 4: GND -> +3.3V
- L58 pad 1: +3.3V -> GND
- L58 pad 2: unconnected-(L58-DOUT-Pad2) -> Net-(L44-DOUT)
- L58 pad 4: GND -> +3.3V
- L6 pad 2: Net-(L6-DOUT) -> /left/LED_DAT
- L7 pad 3: Net-(L6-DOUT) -> Net-(L1-DIN)
- S59 pad A: R_E_2 -> /left/R_E_2
- S59 pad B: R_E_1 -> /left/R_E_1
- S59 pad S1: R_E_S -> /left/R_E_S
- S60 pad A: R_E_2 -> /right/R_E_2
- S60 pad B: R_E_1 -> /right/R_E_1
- S60 pad S1: R_E_S -> /right/R_E_S
- S61 pad 1: VBAT -> /left/VBAT
- S62 pad 1: VBAT -> /right/VBAT
- SW1 pad 1: COL6 -> /left/COL6
- SW10 pad 1: COL3 -> /left/COL3
- SW11 pad 1: COL4 -> /left/COL4
- SW12 pad 1: COL5 -> /left/COL5
- SW13 pad 1: COL6 -> /left/COL6
- SW14 pad 1: COL1 -> /left/COL1
- SW15 pad 1: COL2 -> /left/COL2
- SW16 pad 1: COL3 -> /left/COL3
- SW17 pad 1: COL4 -> /left/COL4
- SW18 pad 1: COL5 -> /left/COL5
- SW19 pad 1: COL6 -> /left/COL6
- SW2 pad 1: COL1 -> /left/COL1
- SW20 pad 1: COL1 -> /left/COL1
- SW21 pad 1: COL2 -> /left/COL2
- SW22 pad 1: COL3 -> /left/COL3
- SW23 pad 1: COL4 -> /left/COL4
- SW24 pad 1: COL5 -> /left/COL5
- SW25 pad 1: COL1 -> /left/COL1
- SW26 pad 1: COL2 -> /left/COL2
- SW27 pad 1: COL3 -> /left/COL3
- SW28 pad 1: COL4 -> /left/COL4
- SW29 pad 1: COL5 -> /left/COL5
- SW3 pad 1: COL2 -> /left/COL2
- SW30 pad 1: COL1 -> /right/COL1
- SW31 pad 1: COL2 -> /right/COL2
- SW32 pad 1: COL3 -> /right/COL3
- SW33 pad 1: COL4 -> /right/COL4
- SW34 pad 1: COL5 -> /right/COL5
- SW35 pad 1: COL6 -> /right/COL6
- SW36 pad 1: COL1 -> /right/COL1
- SW37 pad 1: COL2 -> /right/COL2
- SW38 pad 1: COL3 -> /right/COL3
- SW39 pad 1: COL4 -> /right/COL4
- SW4 pad 1: COL3 -> /left/COL3
- SW40 pad 1: COL5 -> /right/COL5
- SW41 pad 1: COL6 -> /right/COL6
- SW42 pad 1: COL1 -> /right/COL1
- SW43 pad 1: COL2 -> /right/COL2
- SW44 pad 1: COL3 -> /right/COL3
- SW45 pad 1: COL4 -> /right/COL4
- SW46 pad 1: COL5 -> /right/COL5
- SW47 pad 1: COL6 -> /right/COL6
- SW48 pad 1: COL1 -> /right/COL1
- SW49 pad 1: COL2 -> /right/COL2
- SW5 pad 1: COL4 -> /left/COL4
- SW50 pad 1: COL3 -> /right/COL3
- SW51 pad 1: COL4 -> /right/COL4
- SW52 pad 1: COL5 -> /right/COL5
- SW53 pad 1: COL6 -> /right/COL6
- SW54 pad 1: COL1 -> /right/COL1
- SW55 pad 1: COL2 -> /right/COL2
- SW56 pad 1: COL3 -> /right/COL3
- SW57 pad 1: COL4 -> /right/COL4
- SW58 pad 1: COL5 -> /right/COL5
- SW6 pad 1: COL5 -> /left/COL5
- SW7 pad 1: COL6 -> /left/COL6
- SW8 pad 1: COL1 -> /left/COL1
- SW9 pad 1: COL2 -> /left/COL2
- U3 pad 1: unconnected-(U3-P0.06-Pad1) -> /left/ROW1
- U3 pad 10: ROW2 -> /left/COL3
- U3 pad 11: ROW3 -> /left/COL2
- U3 pad 12: ROW4 -> /left/ROW3
- U3 pad 13: VBAT -> /left/VBAT
- U3 pad 17: R_E_S -> /left/COL6
- U3 pad 18: COL6 -> /left/COL1
- U3 pad 19: COL5 -> unconnected-(U3-P0.02-LF-Pad19)
- U3 pad 2: LED_DAT -> /left/LED_DAT
- U3 pad 20: COL4 -> unconnected-(U3-P1.15-LF-Pad20)
- U3 pad 21: COL3 -> unconnected-(U3-P1.13-LF-Pad21)
- U3 pad 22: COL2 -> unconnected-(U3-P1.11-LF-Pad22)
- U3 pad 23: COL1 -> /left/ROW4
- U3 pad 24: ROW5 -> /left/ROW5
- U3 pad 25: unconnected-(U3-P1.01-LF-Pad25) -> /left/R_E_1
- U3 pad 26: unconnected-(U3-P1.02-LF-Pad26) -> /left/R_E_2
- U3 pad 27: unconnected-(U3-P1.07-LF-Pad27) -> /left/R_E_S
- U3 pad 29: VBAT -> /left/VBAT
- U3 pad 5: SDA -> /left/SDA
- U3 pad 6: SCL -> /left/SCL
- U3 pad 7: R_E_1 -> /left/ROW2
- U3 pad 8: R_E_2 -> /left/COL4
- U3 pad 9: ROW1 -> /left/COL5
- U4 pad 1: unconnected-(U4-P0.06-Pad1) -> /right/ROW1
- U4 pad 10: ROW2 -> /right/COL3
- U4 pad 11: ROW3 -> /right/COL2
- U4 pad 12: ROW4 -> /right/ROW3
- U4 pad 13: VBAT -> /right/VBAT
- U4 pad 17: R_E_S -> /right/COL6
- U4 pad 18: COL6 -> /right/COL1
- U4 pad 19: COL5 -> unconnected-(U4-P0.02-LF-Pad19)
- U4 pad 2: LED_DAT -> /right/LED_DAT
- U4 pad 20: COL4 -> unconnected-(U4-P1.15-LF-Pad20)
- U4 pad 21: COL3 -> unconnected-(U4-P1.13-LF-Pad21)
- U4 pad 22: COL2 -> unconnected-(U4-P1.11-LF-Pad22)
- U4 pad 23: COL1 -> /right/ROW4
- U4 pad 24: ROW5 -> /right/ROW5
- U4 pad 25: unconnected-(U4-P1.01-LF-Pad25) -> /right/R_E_1
- U4 pad 26: unconnected-(U4-P1.02-LF-Pad26) -> /right/R_E_2
- U4 pad 27: unconnected-(U4-P1.07-LF-Pad27) -> /right/R_E_S
- U4 pad 29: VBAT -> /right/VBAT
- U4 pad 5: SDA -> /right/SDA
- U4 pad 6: SCL -> /right/SCL
- U4 pad 7: R_E_1 -> /right/ROW2
- U4 pad 8: R_E_2 -> /right/COL4
- U4 pad 9: ROW1 -> /right/COL5
Routing:
- net /left/COL6: track 0.00 -> 197.5 mm
- net /left/COL1: track 0.00 -> 195.7 mm
- net /right/COL5: track 0.00 -> 193.7 mm, vias 0 -> 1
- net /right/COL4: track 0.00 -> 173.0 mm
- net /left/ROW4: track 0.00 -> 165.5 mm, vias 0 -> 1
- net /right/ROW5: track 0.00 -> 164.6 mm, vias 0 -> 3
- net /left/ROW5: track 0.00 -> 163.8 mm, vias 0 -> 1
- net /left/COL2: track 0.00 -> 155.1 mm
- net /right/ROW4: track 0.00 -> 154.3 mm, vias 0 -> 1
- net /left/COL3: track 0.00 -> 138.5 mm
- net /right/COL2: track 0.00 -> 138.0 mm, vias 0 -> 2
- net /right/COL3: track 0.00 -> 134.5 mm, vias 0 -> 2
- net /left/COL4: track 0.00 -> 131.1 mm, vias 0 -> 1
- net /left/ROW3: track 0.00 -> 126.6 mm
- net /left/ROW1: track 0.00 -> 125.1 mm
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Other:
- board size 313.2 x 127.8 mm -> 314.9 x 134 mm
