File: PCB/keeby.kicad_pcb (KiCad board)
At the start: 2 copper layers, 314.9 x 134 mm, 192 parts, among them J1 Conn_01x04_Pin, J2 Conn_01x04_Pin, J3 JST_PH, J4 JST_PH, SW1 SW_Push, SW10 SW_Push, SW11 SW_Push, SW12 SW_Push, SW13 SW_Push, SW14 SW_Push, SW15 SW_Push, SW16 SW_Push, SW17 SW_Push, SW18 SW_Push, SW19 SW_Push, SW2 SW_Push, SW20 SW_Push, SW21 SW_Push, SW22 SW_Push, SW23 SW_Push, SW24 SW_Push, SW25 SW_Push, SW26 SW_Push, SW27 SW_Push, SW28 SW_Push, SW29 SW_Push, SW3 SW_Push, SW30 SW_Push, SW31 SW_Push, SW32 SW_Push, SW33 SW_Push, SW34 SW_Push, SW35 SW_Push, SW36 SW_Push, SW37 SW_Push, SW38 SW_Push, SW39 SW_Push, SW4 SW_Push, SW40 SW_Push, SW41 SW_Push, SW42 SW_Push, SW43 SW_Push, SW44 SW_Push, SW45 SW_Push, SW46 SW_Push, SW47 SW_Push, SW48 SW_Push, SW49 SW_Push, SW5 SW_Push, SW50 SW_Push, SW51 SW_Push, SW52 SW_Push, SW53 SW_Push, SW54 SW_Push, SW55 SW_Push, SW56 SW_Push, SW57 SW_Push, SW58 SW_Push, SW6 SW_Push, SW7 SW_Push, SW8 SW_Push, SW9 SW_Push, U3 SuperMini nRF52840, U4 SuperMini nRF52840

Commit message: addes case
Routing:
- net +3.3V: track 1287.4 -> 557.8 mm, vias 37 -> 14
- net (no net): track 301.8 -> 36.5 mm, vias 8 -> 6
- net Net-(L1-DIN): track 42.6 -> 0.00 mm, vias 2 -> 0
- net Net-(L13-DIN): track 39.3 -> 0.00 mm, vias 2 -> 0
- net /left/LED_DAT: track 34.6 -> 0.00 mm, vias 1 -> 0
- net Net-(L1-DOUT): track 29.9 -> 0.00 mm
- net Net-(L13-DOUT): track 29.9 -> 0.00 mm
- net Net-(L10-DOUT): track 29.6 -> 0.00 mm
- net Net-(L10-DIN): track 29.6 -> 0.00 mm
- net Net-(L11-DIN): track 0.00 -> 22.5 mm, vias 0 -> 2

Commit message: fixing routing again
Parts:
- moved H5 150.5 mm to (56.4, 120.0)
- moved H4 140.1 mm to (295.3, 33.0)
- moved H6 128.4 mm to (305.5, 120.0)
- moved H3 114.2 mm to (66.7, 33.0)
- moved H7 94.1 mm to (144.0, 127.8)
- moved H2 93.7 mm to (238.7, 32.0)
- moved H1 58.2 mm to (123.3, 32.0)
- moved H8 40.9 mm to (218.0, 123.8)
- moved D29 18.9 mm to (156.5, 144.8), turned to 60 degrees
- moved D9 18.9 mm to (101.0, 64.7), turned to 90 degrees
- moved D1 18.9 mm to (62.9, 51.3), turned to 90 degrees
- moved D13 18.9 mm to (62.9, 89.4), turned to 90 degrees
- moved D14 18.9 mm to (81.9, 86.6), turned to 90 degrees
- moved D15 18.9 mm to (101.0, 83.7), turned to 90 degrees
- moved D16 18.9 mm to (120.0, 86.6), turned to 90 degrees
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Routing:
- net +3.3V: track 557.8 -> 0.00 mm, vias 14 -> 0
- net /left/COL6: track 197.5 -> 0.00 mm
- net /left/COL1: track 194.4 -> 0.00 mm, vias 1 -> 0
- net /right/COL5: track 193.7 -> 0.00 mm, vias 1 -> 0
- net /right/COL2: track 177.0 -> 0.00 mm, vias 4 -> 0
- net /right/COL4: track 175.3 -> 0.00 mm, vias 1 -> 0
- net /left/COL2: track 153.8 -> 0.00 mm, vias 1 -> 0
- net /right/COL3: track 145.9 -> 0.00 mm, vias 4 -> 0
- net /left/COL3: track 137.2 -> 0.00 mm, vias 1 -> 0
- net /left/COL4: track 129.8 -> 0.00 mm, vias 2 -> 0
- net /left/COL5: track 123.8 -> 0.00 mm, vias 2 -> 0
- net /right/COL1: track 110.4 -> 0.00 mm, vias 2 -> 0
- net /left/ROW5: track 163.8 -> 85.0 mm, vias 1 -> 0
- net /right/ROW5: track 164.6 -> 94.7 mm, vias 3 -> 0
- net /left/ROW4: track 165.5 -> 102.0 mm, vias 1 -> 0
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Other:
- board size 314.9 x 134 mm -> 313.2 x 127.9 mm

Commit message: routed left
Routing:
- net +3.3V: track 0.00 -> 729.6 mm, vias 0 -> 19
- net /left/COL1: track 0.00 -> 221.7 mm, vias 0 -> 5
- net /left/COL2: track 0.00 -> 204.9 mm, vias 0 -> 5
- net /left/COL6: track 0.00 -> 197.9 mm
- net /left/COL3: track 0.00 -> 151.6 mm
- net /left/COL4: track 0.00 -> 141.4 mm, vias 0 -> 1
- net /left/COL5: track 0.00 -> 136.4 mm, vias 0 -> 2
- net /left/ROW5: track 85.0 -> 170.4 mm, vias 0 -> 1
- net /right/VBAT: track 0.00 -> 67.8 mm, vias 0 -> 1
- net /left/R_E_1: track 0.00 -> 62.4 mm
- net /left/ROW4: track 102.0 -> 163.3 mm, vias 0 -> 1
- net /right/COL6: track 0.00 -> 60.2 mm
- net /right/COL5: track 0.00 -> 60.1 mm
- net /right/COL2: track 0.00 -> 60.1 mm
- net /right/COL1: track 0.00 -> 59.8 mm
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
Commit message: routed full
Routing:
- net +3.3V: track 729.6 -> 1413.6 mm, vias 19 -> 25
- net /right/COL5: track 60.1 -> 234.3 mm, vias 0 -> 6
- net /right/COL6: track 60.2 -> 209.8 mm, vias 0 -> 5
- net /right/COL4: track 59.8 -> 204.8 mm, vias 0 -> 6
- net /right/COL3: track 59.8 -> 163.0 mm, vias 0 -> 4
- net /right/COL1: track 59.8 -> 158.0 mm, vias 0 -> 2
- net /right/COL2: track 60.1 -> 157.5 mm, vias 0 -> 4
- net /right/R_E_2: track 0.00 -> 65.5 mm, vias 0 -> 1
- net /right/ROW5: track 94.5 -> 159.2 mm, vias 0 -> 2
- net /right/ROW4: track 99.3 -> 156.2 mm, vias 0 -> 2
- net /right/R_E_1: track 0.00 -> 53.4 mm
- net /right/R_E_S: track 0.00 -> 38.3 mm, vias 0 -> 1
- net /right/SDA: track 0.00 -> 30.4 mm
- net /right/SCL: track 0.00 -> 28.1 mm
- net Net-(L35-DOUT): track 33.5 -> 27.6 mm
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