File: PCB/half.kicad_sch (KiCad schematic)
At the start: 95 parts, among them J3 JST_PH, SW1 SW_Push, SW10 SW_Push, SW11 SW_Push, SW12 SW_Push, SW13 SW_Push, SW14 SW_Push, SW15 SW_Push, SW16 SW_Push, SW17 SW_Push, SW18 SW_Push, SW19 SW_Push, SW2 SW_Push, SW20 SW_Push, SW21 SW_Push, SW22 SW_Push, SW23 SW_Push, SW24 SW_Push, SW25 SW_Push, SW26 SW_Push, SW27 SW_Push, SW28 SW_Push, SW29 SW_Push, SW3 SW_Push, SW4 SW_Push, SW5 SW_Push, SW59 RotaryEncoder_Switch, SW6 SW_Push, SW61 SW_SPDT, SW7 SW_Push, SW8 SW_Push, SW9 SW_Push, U3 SuperMini nRF52840

Commit message: prepared outline
Parts:
- S61: renamed from SW61; value SW_SPDT -> S_SPDT
- renumbered SW59 to S59, SW6 to SW1, SW9 to SW10, SW10 to SW11, SW11 to SW12, SW18 to SW13, SW13 to SW14, SW14 to SW15, SW15 to SW16, SW16 to SW17, SW17 to SW18, SW24 to SW19, SW1 to SW2, SW19 to SW20, SW20 to SW21, SW21 to SW22, SW22 to SW23, SW23 to SW24, SW2 to SW3, SW3 to SW4, SW4 to SW5, SW5 to SW6, SW12 to SW7, SW7 to SW8, SW8 to SW9
Changed lines of the file:
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@@
 		(dnp no)
 		(fields_autoplaced yes)
-		(property "Reference" "SW61"
-			(at 189.23 92.71 0)
+		(property "Reference" "S61"
+			(at 189.23 74.93 0)
 			(effects
 				(font
@@
 			)
 		)
-		(property "Value" "SW_SPDT"
-			(at 189.23 90.17 0)
+		(property "Value" "S_SPDT"
+			(at 189.23 77.47 0)
 			(effects
 				(font
@@
 			(project ""
 				(path "/fade6638-4e22-4fdd-8807-944beeb130ad/0032fa72-ac59-4218-be72-f997fa7d8d03"
-					(reference "SW62")
+					(reference "S62")
 					(unit 1)
 				)
 				(path "/fade6638-4e22-4fdd-8807-944beeb130ad/7560e8d7-2115-4052-abf3-3690798ba6d5"
-					(reference "SW61")
+					(reference "S61")
 					(unit 1)
 				)
@@
 		(dnp no)
 		(fields_autoplaced yes)
-		(property "Reference" "SW11"
+		(property "Reference" "SW12"
 			(at 123.19 106.68 0)
 			(effects
@@
 				)
 				(path "/fade6638-4e22-4fdd-8807-944beeb130ad/7560e8d7-2115-4052-abf3-3690798ba6d5"
-					(reference "SW11")
+					(reference "SW12")
 					(unit 1)
 				)
@@
 		(dnp no)
 		(fields_autoplaced yes)
-		(property "Reference" "SW3"
+		(property "Reference" "SW4"
 			(at 80.01 87.63 0)
 			(effects
@@
 				)
 				(path "/fade6638-4e22-4fdd-8807-944beeb130ad/7560e8d7-2115-4052-abf3-3690798ba6d5"
-					(reference "SW3")
+					(reference "SW4")
 					(unit 1)
 				)
@@
 		(dnp no)
 		(fields_autoplaced yes)
-		(property "Reference" "SW15"
+		(property "Reference" "SW16"
 			(at 80.01 125.73 0)
 			(effects
@@
 				)
 				(path "/fade6638-4e22-4fdd-8807-944beeb130ad/7560e8d7-2115-4052-abf3-3690798ba6d5"
-					(reference "SW15")
+					(reference "SW16")
 					(unit 1)
 				)
@@
 		(dnp no)
 		(fields_autoplaced yes)
-		(property "Reference" "SW20"
+		(property "Reference" "SW21"
 			(at 58.42 144.78 0)
 			(effects
@@
 				)
 				(path "/fade6638-4e22-4fdd-8807-944beeb130ad/7560e8d7-2115-4052-abf3-3690798ba6d5"
-					(reference "SW20")
+					(reference "SW21")
 					(unit 1)
 				)
@@
 		(dnp no)
 		(fields_autoplaced yes)
-		(property "Reference" "SW4"
+		(property "Reference" "SW5"
 			(at 101.6 87.63 0)
 			(effects
@@
 				)
 				(path "/fade6638-4e22-4fdd-8807-944beeb130ad/7560e8d7-2115-4052-abf3-3690798ba6d5"
-					(reference "SW4")
+					(reference "SW5")
 					(unit 1)
 				)
@@
 		(dnp no)
 		(fields_autoplaced yes)
-		(property "Reference" "SW16"
+		(property "Reference" "SW17"
 			(at 101.6 125.73 0)
 			(effects
@@
 				)
 				(path "/fade6638-4e22-4fdd-8807-944beeb130ad/7560e8d7-2115-4052-abf3-3690798ba6d5"
-					(reference "SW16")
+					(reference "SW17")
 					(unit 1)
 				)
@@
 		(dnp no)
 		(fields_autoplaced yes)
-		(property "Reference" "SW18"
+		(property "Reference" "SW13"
 			(at 144.78 125.73 0)
 			(effects
@@
 				)
 				(path "/fade6638-4e22-4fdd-8807-944beeb130ad/7560e8d7-2115-4052-abf3-3690798ba6d5"
-					(reference "SW18")
+					(reference "SW13")
 					(unit 1)
 				)
@@
 		(dnp no)
 		(fields_autoplaced yes)
-		(property "Reference" "SW9"
+		(property "Reference" "SW10"
 			(at 80.01 106.68 0)
 			(effects
@@
 				)
 				(path "/fade6638-4e22-4fdd-8807-944beeb130ad/7560e8d7-2115-4052-abf3-3690798ba6d5"
-					(reference "SW9")
+					(reference "SW10")
 					(unit 1)
 				)
@@
 		(dnp no)
 		(fields_autoplaced yes)
-		(property "Reference" "SW24"
+		(property "Reference" "SW19"
 			(at 144.78 144.78 0)
 			(effects
@@
 				)
 				(path "/fade6638-4e22-4fdd-8807-944beeb130ad/7560e8d7-2115-4052-abf3-3690798ba6d5"
-					(reference "SW24")
+					(reference "SW19")
 					(unit 1)
 				)
@@
 		(dnp no)
 		(fields_autoplaced yes)
-		(property "Reference" "SW14"
+		(property "Reference" "SW15"
 			(at 58.42 125.73 0)
 			(effects
@@
 				)
 				(path "/fade6638-4e22-4fdd-8807-944beeb130ad/7560e8d7-2115-4052-abf3-3690798ba6d5"
-					(reference "SW14")
+					(reference "SW15")
 					(unit 1)
 				)
@@
 		(dnp no)
 		(fields_autoplaced yes)
-		(property "Reference" "SW12"
+		(property "Reference" "SW7"
 			(at 144.78 106.68 0)
 			(effects
@@
 				)
 				(path "/fade6638-4e22-4fdd-8807-944beeb130ad/7560e8d7-2115-4052-abf3-3690798ba6d5"
-					(reference "SW12")
+					(reference "SW7")
 					(unit 1)
 				)
@@
 		(dnp no)
 		(fields_autoplaced yes)
-		(property "Reference" "SW13"
+		(property "Reference" "SW14"
 			(at 36.83 125.73 0)
 			(effects
@@
 				)
 				(path "/fade6638-4e22-4fdd-8807-944beeb130ad/7560e8d7-2115-4052-abf3-3690798ba6d5"
-					(reference "SW13")
+					(reference "SW14")
 					(unit 1)
 				)
@@
 		(dnp no)
 		(fields_autoplaced yes)
-		(property "Reference" "SW22"
+		(property "Reference" "SW23"
 			(at 101.6 144.78 0)
 			(effects
@@
 				)
 				(path "/fade6638-4e22-4fdd-8807-944beeb130ad/7560e8d7-2115-4052-abf3-3690798ba6d5"
-					(reference "SW22")
+					(reference "SW23")
 					(unit 1)
 				)
@@
 		(dnp no)
 		(fields_autoplaced yes)
-		(property "Reference" "SW23"
+		(property "Reference" "SW24"
 			(at 123.19 144.78 0)
 			(effects
@@
 				)
 				(path "/fade6638-4e22-4fdd-8807-944beeb130ad/7560e8d7-2115-4052-abf3-3690798ba6d5"
-					(reference "SW23")
+					(reference "SW24")
 					(unit 1)
 				)
@@
 		(dnp no)
 		(fields_autoplaced yes)
-		(property "Reference" "SW8"
+		(property "Reference" "SW9"
 			(at 58.42 106.68 0)
 			(effects
@@
 				)
 				(path "/fade6638-4e22-4fdd-8807-944beeb130ad/7560e8d7-2115-4052-abf3-3690798ba6d5"
-					(reference "SW8")
+					(reference "SW9")
 					(unit 1)
 				)
@@
 		(dnp no)
 		(fields_autoplaced yes)
-		(property "Reference" "SW59"
+		(property "Reference" "S59"
 			(at 148.59 168.91 0)
 			(effects
@@
 			(project ""
 				(path "/fade6638-4e22-4fdd-8807-944beeb130ad/0032fa72-ac59-4218-be72-f997fa7d8d03"
-					(reference "SW60")
+					(reference "S60")
 					(unit 1)
 				)
 				(path "/fade6638-4e22-4fdd-8807-944beeb130ad/7560e8d7-2115-4052-abf3-3690798ba6d5"
-					(reference "SW59")
+					(reference "S59")
 					(unit 1)
 				)
@@
 		(dnp no)
 		(fields_autoplaced yes)
-		(property "Reference" "SW5"
+		(property "Reference" "SW6"
 			(at 123.19 87.63 0)
 			(effects
@@
 				)
 				(path "/fade6638-4e22-4fdd-8807-944beeb130ad/7560e8d7-2115-4052-abf3-3690798ba6d5"
-					(reference "SW5")
+					(reference "SW6")
 					(unit 1)
 				)
@@
 		(dnp no)
 		(fields_autoplaced yes)
-		(property "Reference" "SW19"
+		(property "Reference" "SW20"
 			(at 36.83 144.78 0)
 			(effects
@@
 				)
 				(path "/fade6638-4e22-4fdd-8807-944beeb130ad/7560e8d7-2115-4052-abf3-3690798ba6d5"
-					(reference "SW19")
+					(reference "SW20")
 					(unit 1)
 				)
@@
 		(dnp no)
 		(fields_autoplaced yes)
-		(property "Reference" "SW10"
+		(property "Reference" "SW11"
 			(at 101.6 106.68 0)
 			(effects
@@
 				)
 				(path "/fade6638-4e22-4fdd-8807-944beeb130ad/7560e8d7-2115-4052-abf3-3690798ba6d5"
-					(reference "SW10")
+					(reference "SW11")
 					(unit 1)
 				)
@@
 		(dnp no)
 		(fields_autoplaced yes)
-		(property "Reference" "SW6"
+		(property "Reference" "SW1"
 			(at 144.78 87.63 0)
 			(effects
@@
 				)
 				(path "/fade6638-4e22-4fdd-8807-944beeb130ad/7560e8d7-2115-4052-abf3-3690798ba6d5"
-					(reference "SW6")
+					(reference "SW1")
 					(unit 1)
 				)
@@
 		(dnp no)
 		(fields_autoplaced yes)
-		(property "Reference" "SW17"
+		(property "Reference" "SW18"
 			(at 123.19 125.73 0)
 			(effects
@@
 				)
 				(path "/fade6638-4e22-4fdd-8807-944beeb130ad/7560e8d7-2115-4052-abf3-3690798ba6d5"
-					(reference "SW17")
+					(reference "SW18")
 					(unit 1)
 				)
@@
 		(dnp no)
 		(fields_autoplaced yes)
-		(property "Reference" "SW21"
+		(property "Reference" "SW22"
 			(at 80.01 144.78 0)
 			(effects
@@
 				)
 				(path "/fade6638-4e22-4fdd-8807-944beeb130ad/7560e8d7-2115-4052-abf3-3690798ba6d5"
-					(reference "SW21")
+					(reference "SW22")
 					(unit 1)
 				)
@@
 		(dnp no)
 		(fields_autoplaced yes)
-		(property "Reference" "SW1"
+		(property "Reference" "SW2"
 			(at 36.83 87.63 0)
 			(effects
@@
 				)
 				(path "/fade6638-4e22-4fdd-8807-944beeb130ad/7560e8d7-2115-4052-abf3-3690798ba6d5"
-					(reference "SW1")
+					(reference "SW2")
 					(unit 1)
 				)
@@
 		(dnp no)
 		(fields_autoplaced yes)
-		(property "Reference" "SW7"
+		(property "Reference" "SW8"
 			(at 36.83 106.68 0)
 			(effects
@@
 				)
 				(path "/fade6638-4e22-4fdd-8807-944beeb130ad/7560e8d7-2115-4052-abf3-3690798ba6d5"
-					(reference "SW7")
+					(reference "SW8")
 					(unit 1)
 				)
@@
 		(dnp no)
 		(fields_autoplaced yes)
-		(property "Reference" "SW2"
+		(property "Reference" "SW3"
 			(at 58.42 87.63 0)
 			(effects
@@
 				)
 				(path "/fade6638-4e22-4fdd-8807-944beeb130ad/7560e8d7-2115-4052-abf3-3690798ba6d5"
-					(reference "SW2")
+					(reference "SW3")
 					(unit 1)
 				)

Commit message: fixing leds
Parts:
- L1, L10, L11, L12, L13, L14, L15, L16, L17, L18, L19, L2, L20, L21, L22, L23, L24, L25, L26, L27, L28, L29, L3, L4, L5, L6, L7, L8, L9: value SK6812MINI -> SK6812-MINI-E
Connections:
- net +3.3V: now also L16.4 (VSS), L17.4 (VSS), L18.4 (VSS), L19.4 (VSS), L20.4 (VSS), L21.4 (VSS), L22.4 (VSS), L23.4 (VSS), L24.4 (VSS), L25.4 (VSS), L26.4 (VSS), L27.4 (VSS), L28.4 (VSS), L29.4 (VSS); no longer L16.1 (VDD), L17.1 (VDD), L18.1 (VDD), L19.1 (VDD), L20.1 (VDD), L21.1 (VDD), L22.1 (VDD), L23.1 (VDD), L24.1 (VDD), L25.1 (VDD), L26.1 (VDD), L27.1 (VDD), L28.1 (VDD), L29.1 (VDD)
- net COL1: now also U3.18 (P0.29-LF); no longer U3.23 (P0.10-LF)
- net COL2: now also U3.11 (P1.04-LF); no longer U3.22 (P1.11-LF)
- net COL3: now also U3.10 (P0.11); no longer U3.21 (P1.13-LF)
- net COL4: now also U3.8 (P0.24); no longer U3.20 (P1.15-LF)
- net COL5: now also U3.9 (P1.00); no longer U3.19 (P0.02-LF)
- net COL6: now also U3.17 (P0.31-LF); no longer U3.18 (P0.29-LF)
- net GND: now also L16.1 (VDD), L17.1 (VDD), L18.1 (VDD), L19.1 (VDD), L20.1 (VDD), L21.1 (VDD), L22.1 (VDD), L23.1 (VDD), L24.1 (VDD), L25.1 (VDD), L26.1 (VDD), L27.1 (VDD), L28.1 (VDD), L29.1 (VDD); no longer L16.4 (VSS), L17.4 (VSS), L18.4 (VSS), L19.4 (VSS), L20.4 (VSS), L21.4 (VSS), L22.4 (VSS), L23.4 (VSS), L24.4 (VSS), L25.4 (VSS), L26.4 (VSS), L27.4 (VSS), L28.4 (VSS), L29.4 (VSS)
- net LED_DAT: now also L6.2 (DOUT); no longer L1.3 (DIN)
- net ROW1: now also U3.1 (P0.06); no longer U3.9 (P1.00)
- net ROW2: now also U3.7 (P0.22); no longer U3.10 (P0.11)
- net ROW3: now also U3.12 (P1.06-LF); no longer U3.11 (P1.04-LF)
- net ROW4: now also U3.23 (P0.10-LF); no longer U3.12 (P1.06-LF)
- net R_E_1: now also U3.25 (P1.01-LF); no longer U3.7 (P0.22)
- net R_E_2: now also U3.26 (P1.02-LF); no longer U3.8 (P0.24)
- net R_E_S: now also U3.27 (P1.07-LF); no longer U3.17 (P0.31-LF)
- net at L18.2 (DOUT): now also L17.3 (DIN); no longer L19.3 (DIN)
- net at L18.3 (DIN): now also L12.2 (DOUT); no longer L17.2 (DOUT)
- net at L24.2 (DOUT): now also L23.3 (DIN); no longer L25.3 (DIN)
- net at L24.3 (DIN): now also L29.3 (DIN); no longer L23.2 (DOUT)
- net at L27.2 (DOUT): now also L26.3 (DIN); no longer L28.3 (DIN)
- net at L27.3 (DIN): now also L28.2 (DOUT); no longer L26.2 (DOUT)
- net at L7.3 (DIN): now also L1.3 (DIN); no longer L6.2 (DOUT)
- net at L13.3 (DIN): now also L19.2 (DOUT); no longer L12.2 (DOUT)
- net at L15.2 (DOUT): now also L16.2 (DOUT); no longer L16.3 (DIN)
- net at L29.2 (DOUT): now also L28.3 (DIN)
- net at L25.2 (DOUT): no longer L26.3 (DIN)
- net at L22.2 (DOUT): now also L21.3 (DIN); no longer L23.3 (DIN)
- net at L22.3 (DIN): now also L23.2 (DOUT); no longer L21.2 (DOUT)
- net at L20.3 (DIN): now also L21.2 (DOUT); no longer L19.2 (DOUT)
- net at L20.2 (DOUT): now also L19.3 (DIN); no longer L21.3 (DIN)
- new net: L25.3 (DIN), L26.2 (DOUT)
- new net: L16.3 (DIN), L17.2 (DOUT)
Other:
- moved on the sheet: D1, D10, D11, D12, D13, D14, D15, D16, D17, D18, D19, D2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

Commit message: routing
Connections:
- net +3.3V: now also L16.1 (VDD), L17.1 (VDD), L18.1 (VDD), L19.1 (VDD), L20.1 (VDD), L21.1 (VDD), L22.1 (VDD), L23.1 (VDD), L24.1 (VDD), L25.1 (VDD), L26.1 (VDD), L27.1 (VDD), L28.1 (VDD), L29.1 (VDD); no longer L16.4 (VSS), L17.4 (VSS), L18.4 (VSS), L19.4 (VSS), L20.4 (VSS), L21.4 (VSS), L22.4 (VSS), L23.4 (VSS), L24.4 (VSS), L25.4 (VSS), L26.4 (VSS), L27.4 (VSS), L28.4 (VSS), L29.4 (VSS)
- net GND: now also L16.4 (VSS), L17.4 (VSS), L18.4 (VSS), L19.4 (VSS), L20.4 (VSS), L21.4 (VSS), L22.4 (VSS), L23.4 (VSS), L24.4 (VSS), L25.4 (VSS), L26.4 (VSS), L27.4 (VSS), L28.4 (VSS), L29.4 (VSS); no longer L16.1 (VDD), L17.1 (VDD), L18.1 (VDD), L19.1 (VDD), L20.1 (VDD), L21.1 (VDD), L22.1 (VDD), L23.1 (VDD), L24.1 (VDD), L25.1 (VDD), L26.1 (VDD), L27.1 (VDD), L28.1 (VDD), L29.1 (VDD)
- net at L18.2 (DOUT): now also L12.2 (DOUT); no longer L17.3 (DIN)
- net at L18.3 (DIN): now also L17.2 (DOUT); no longer L12.2 (DOUT)
- net at L24.2 (DOUT): now also L29.2 (DOUT); no longer L23.3 (DIN)
- net at L24.3 (DIN): now also L23.2 (DOUT); no longer L29.3 (DIN)
- net at L27.2 (DOUT): now also L28.3 (DIN); no longer L26.3 (DIN)
- net at L27.3 (DIN): now also L26.2 (DOUT); no longer L28.2 (DOUT)
- net at L13.3 (DIN): now also L19.3 (DIN); no longer L19.2 (DOUT)
- net at L15.2 (DOUT): now also L16.3 (DIN); no longer L16.2 (DOUT)
- net at L25.2 (DOUT): now also L26.3 (DIN)
- net at L25.3 (DIN): no longer L26.2 (DOUT)
- net at L22.2 (DOUT): now also L23.3 (DIN); no longer L21.3 (DIN)
- net at L22.3 (DIN): now also L21.2 (DOUT); no longer L23.2 (DOUT)
- net at L20.2 (DOUT): now also L21.3 (DIN); no longer L19.3 (DIN)
- net at L20.3 (DIN): now also L19.2 (DOUT); no longer L21.2 (DOUT)
- new net: L28.2 (DOUT), L29.3 (DIN)
- new net: L16.2 (DOUT), L17.3 (DIN)
Other:
- moved on the sheet: L16, L17, L18, L19, L20, L21, L22, L23, L24, L25, L26, L27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
Changed lines of the file:
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@@
 	(symbol
 		(lib_id "marbastlib-various:SK6812MINI-E")
-		(at 342.9 113.03 180)
+		(at 342.9 113.03 0)
 		(unit 1)
 		(exclude_from_sim no)
@@
 		(dnp no)
 		(property "Reference" "L18"
-			(at 342.9 124.968 0)
+			(at 342.9 101.092 0)
 			(effects
 				(font
@@
 		)
 		(property "Value" "SK6812-MINI-E"
-			(at 342.9 122.428 0)
+			(at 342.9 103.632 0)
 			(effects
 				(font
@@
 	(symbol
 		(lib_id "marbastlib-various:SK6812MINI-E")
-		(at 341.63 140.97 180)
+		(at 341.63 140.97 0)
 		(unit 1)
 		(exclude_from_sim no)
@@
 		(dnp no)
 		(property "Reference" "L24"
-			(at 341.63 152.908 0)
+			(at 341.63 129.032 0)
 			(effects
 				(font
@@
 		)
 		(property "Value" "SK6812-MINI-E"
-			(at 341.63 150.368 0)
+			(at 341.63 131.572 0)
 			(effects
 				(font
@@
 	(symbol
 		(lib_id "marbastlib-various:SK6812MINI-E")
-		(at 270.51 168.91 180)
+		(at 270.51 168.91 0)
 		(unit 1)
 		(exclude_from_sim no)
@@
 		(dnp no)
 		(property "Reference" "L27"
-			(at 270.51 155.448 0)
+			(at 270.51 156.972 0)
 			(effects
 				(font
@@
 		)
 		(property "Value" "SK6812-MINI-E"
-			(at 270.51 157.734 0)
+			(at 270.51 159.512 0)
 			(effects
 				(font
@@
 	(symbol
 		(lib_id "marbastlib-various:SK6812MINI-E")
-		(at 318.77 168.91 180)
+		(at 318.77 168.91 0)
 		(unit 1)
 		(exclude_from_sim no)
@@
 		(dnp no)
 		(property "Reference" "L29"
-			(at 318.77 155.448 0)
+			(at 318.77 156.972 0)
 			(effects
 				(font
@@
 		)
 		(property "Value" "SK6812-MINI-E"
-			(at 318.77 157.734 0)
+			(at 318.77 159.512 0)
 			(effects
 				(font
@@
 	(symbol
 		(lib_id "marbastlib-various:SK6812MINI-E")
-		(at 222.25 168.91 180)
+		(at 222.25 168.91 0)
 		(unit 1)
 		(exclude_from_sim no)
@@
 		(dnp no)
 		(property "Reference" "L25"
-			(at 222.25 180.848 0)
+			(at 222.25 156.972 0)
 			(effects
 				(font
@@
 		)
 		(property "Value" "SK6812-MINI-E"
-			(at 222.25 178.308 0)
+			(at 222.25 159.512 0)
 			(effects
 				(font
@@
 	(symbol
 		(lib_id "marbastlib-various:SK6812MINI-E")
-		(at 318.77 113.03 180)
+		(at 318.77 113.03 0)
 		(unit 1)
 		(exclude_from_sim no)
@@
 		(dnp no)
 		(property "Reference" "L17"
-			(at 318.77 124.968 0)
+			(at 318.77 101.092 0)
 			(effects
 				(font
@@
 		)
 		(property "Value" "SK6812-MINI-E"
-			(at 318.77 122.428 0)
+			(at 318.77 103.632 0)
 			(effects
 				(font
@@
 	(symbol
 		(lib_id "marbastlib-various:SK6812MINI-E")
-		(at 294.64 140.97 180)
+		(at 294.64 140.97 0)
 		(unit 1)
 		(exclude_from_sim no)
@@
 		(dnp no)
 		(property "Reference" "L22"
-			(at 294.64 152.908 0)
+			(at 294.64 129.032 0)
 			(effects
 				(font
@@
 		)
 		(property "Value" "SK6812-MINI-E"
-			(at 294.64 150.368 0)
+			(at 294.64 131.572 0)
 			(effects
 				(font
@@
 	(symbol
 		(lib_id "marbastlib-various:SK6812MINI-E")
-		(at 245.11 168.91 180)
+		(at 245.11 168.91 0)
 		(unit 1)
 		(exclude_from_sim no)
@@
 		(dnp no)
 		(property "Reference" "L26"
-			(at 245.11 180.848 0)
+			(at 245.11 156.972 0)
 			(effects
 				(font
@@
 		)
 		(property "Value" "SK6812-MINI-E"
-			(at 245.11 178.308 0)
+			(at 245.11 159.512 0)
 			(effects
 				(font
@@
 	(symbol
 		(lib_id "marbastlib-various:SK6812MINI-E")
-		(at 294.64 168.91 180)
+		(at 294.64 168.91 0)
 		(unit 1)
 		(exclude_from_sim no)
@@
 		(dnp no)
 		(property "Reference" "L28"
-			(at 294.64 155.448 0)
+			(at 294.64 156.972 0)
 			(effects
 				(font
@@
 		)
 		(property "Value" "SK6812-MINI-E"
-			(at 294.64 157.734 0)
+			(at 294.64 159.512 0)
 			(effects
 				(font
@@
 	(symbol
 		(lib_id "marbastlib-various:SK6812MINI-E")
-		(at 222.25 140.97 180)
+		(at 222.25 140.97 0)
 		(unit 1)
 		(exclude_from_sim no)
@@
 		(dnp no)
 		(property "Reference" "L19"
-			(at 222.25 152.908 0)
+			(at 222.25 129.032 0)
 			(effects
 				(font
@@
 		)
 		(property "Value" "SK6812-MINI-E"
-			(at 222.25 150.368 0)
+			(at 222.25 131.572 0)
 			(effects
 				(font
@@
 	(symbol
 		(lib_id "marbastlib-various:SK6812MINI-E")
-		(at 294.64 113.03 180)
+		(at 294.64 113.03 0)
 		(unit 1)
 		(exclude_from_sim no)
@@
 		(dnp no)
 		(property "Reference" "L16"
-			(at 294.64 124.968 0)
+			(at 294.64 101.092 0)
 			(effects
 				(font
@@
 		)
 		(property "Value" "SK6812-MINI-E"
-			(at 294.64 122.428 0)
+			(at 294.64 103.632 0)
 			(effects
 				(font
@@
 	(symbol
 		(lib_id "marbastlib-various:SK6812MINI-E")
-		(at 317.5 140.97 180)
+		(at 317.5 140.97 0)
 		(unit 1)
 		(exclude_from_sim no)
@@
 		(dnp no)
 		(property "Reference" "L23"
-			(at 317.5 152.908 0)
+			(at 317.5 129.032 0)
 			(effects
 				(font
@@
 		)
 		(property "Value" "SK6812-MINI-E"
-			(at 317.5 150.368 0)
+			(at 317.5 131.572 0)
 			(effects
 				(font
@@
 	(symbol
 		(lib_id "marbastlib-various:SK6812MINI-E")
-		(at 246.38 140.97 180)
+		(at 246.38 140.97 0)
 		(unit 1)
 		(exclude_from_sim no)
@@
 		(dnp no)
 		(property "Reference" "L20"
-			(at 246.38 152.908 0)
+			(at 246.38 129.032 0)
 			(effects
 				(font
@@
 		)
 		(property "Value" "SK6812-MINI-E"
-			(at 246.38 150.368 0)
+			(at 246.38 131.572 0)
 			(effects
 				(font
@@
 	(symbol
 		(lib_id "marbastlib-various:SK6812MINI-E")
-		(at 270.51 140.97 180)
+		(at 270.51 140.97 0)
 		(unit 1)
 		(exclude_from_sim no)
@@
 		(dnp no)
 		(property "Reference" "L21"
-			(at 270.51 152.908 0)
+			(at 270.51 129.032 0)
 			(effects
 				(font
@@
 		)
 		(property "Value" "SK6812-MINI-E"
-			(at 270.51 150.368 0)
+			(at 270.51 131.572 0)
 			(effects
 				(font

Commit message: addes case
Connections:
- net LED_DAT: now also L6.3 (DIN); no longer L6.2 (DOUT)
- net at L18.2 (DOUT): now also L17.3 (DIN); no longer L12.2 (DOUT)
- net at L18.3 (DIN): now also L12.3 (DIN); no longer L17.2 (DOUT)
- net at L24.2 (DOUT): now also L23.3 (DIN); no longer L29.2 (DOUT)
- net at L24.3 (DIN): now also L29.3 (DIN); no longer L23.2 (DOUT)
- net at L2.2 (DOUT): now also L1.3 (DIN); no longer L3.3 (DIN)
- net at L2.3 (DIN): now also L3.2 (DOUT); no longer L1.2 (DOUT)
- net at L7.3 (DIN): now also L8.2 (DOUT); no longer L1.3 (DIN)
- net at L5.2 (DOUT): now also L4.3 (DIN); no longer L6.3 (DIN)
- net at L5.3 (DIN): now also L6.2 (DOUT); no longer L4.2 (DOUT)
- net at L11.2 (DOUT): now also L10.3 (DIN); no longer L12.3 (DIN)
- net at L11.3 (DIN): now also L12.2 (DOUT); no longer L10.2 (DOUT)
- net at L27.2 (DOUT): now also L26.3 (DIN); no longer L28.3 (DIN)
- net at L27.3 (DIN): now also L28.2 (DOUT); no longer L26.2 (DOUT)
- net at L9.2 (DOUT): now also L8.3 (DIN); no longer L10.3 (DIN)
- net at L9.3 (DIN): now also L10.2 (DOUT); no longer L8.2 (DOUT)
- net at L7.2 (DOUT): now also L1.2 (DOUT); no longer L8.3 (DIN)
- net at L13.2 (DOUT): now also L19.2 (DOUT); no longer L14.3 (DIN)
- net at L13.3 (DIN): now also L14.2 (DOUT); no longer L19.3 (DIN)
- net at L15.2 (DOUT): now also L14.3 (DIN); no longer L16.3 (DIN)
- net at L15.3 (DIN): now also L16.2 (DOUT); no longer L14.2 (DOUT)
- net at L25.2 (DOUT): no longer L26.3 (DIN)
- net at L25.3 (DIN): now also L26.2 (DOUT)
- net at L22.2 (DOUT): now also L21.3 (DIN); no longer L23.3 (DIN)
- net at L22.3 (DIN): now also L23.2 (DOUT); no longer L21.2 (DOUT)
- net at L20.3 (DIN): now also L21.2 (DOUT); no longer L19.2 (DOUT)
- net at L20.2 (DOUT): now also L19.3 (DIN); no longer L21.3 (DIN)
- new net: L28.3 (DIN), L29.2 (DOUT)
- new net: L3.3 (DIN), L4.2 (DOUT)
- new net: L16.3 (DIN), L17.2 (DOUT)
Other:
- moved on the sheet: L1, L10, L11, L12, L13, L14, L15, L16, L17, L18, L19, L2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

Commit message: added decoupling capacitors
Parts:
- added C1, C10, C11, C12, C13, C14, C15, C16, C17, C18, C19, C2, C20, C21, C22, C23, C24, C25, C26, C27, C28, C29, C3, C4, C5, C6, C7, C8, C9: C_Small, symbol Device:C_Small
Connections:
- net +3.3V: now also C1.1, C10.2, C11.2, C12.2, C13.1, C14.1, C15.1, C16.1, C17.1, C18.1, C19.2, C2.1, C20.2, C21.2, C22.2, C23.2, C24.2, C25.1, C26.1, C27.1, C28.1, C29.1, C3.1, C4.1, C5.1, C6.1, C7.2, C8.2, C9.2
- net GND: now also C1.2, C10.1, C11.1, C12.1, C13.2, C14.2, C15.2, C16.2, C17.2, C18.2, C19.1, C2.2, C20.1, C21.1, C22.1, C23.1, C24.1, C25.2, C26.2, C27.2, C28.2, C29.2, C3.2, C4.2, C5.2, C6.2, C7.1, C8.1, C9.1
- net at L18.3 (DIN): now also L12.2 (DOUT); no longer L12.3 (DIN)
- net at L24.2 (DOUT): now also L29.3 (DIN); no longer L23.3 (DIN)
- net at L24.3 (DIN): now also L23.2 (DOUT); no longer L29.3 (DIN)
- net at L1.2 (DOUT): now also L7.3 (DIN); no longer L7.2 (DOUT)
- net at L11.2 (DOUT): now also L12.3 (DIN); no longer L10.3 (DIN)
- net at L11.3 (DIN): now also L10.2 (DOUT); no longer L12.2 (DOUT)
- net at L9.2 (DOUT): now also L10.3 (DIN); no longer L8.3 (DIN)
- net at L9.3 (DIN): now also L8.2 (DOUT); no longer L10.2 (DOUT)
- net at L13.2 (DOUT): now also L19.3 (DIN); no longer L19.2 (DOUT)
- net at L22.2 (DOUT): now also L23.3 (DIN); no longer L21.3 (DIN)
- net at L22.3 (DIN): now also L21.2 (DOUT); no longer L23.2 (DOUT)
- net at L20.2 (DOUT): now also L21.3 (DIN); no longer L19.3 (DIN)
- net at L20.3 (DIN): now also L19.2 (DOUT); no longer L21.2 (DOUT)
- new net: L7.2 (DOUT), L8.3 (DIN)
Other:
- moved on the sheet: L1, L10, L11, L12, L13, L14, L15, L16, L17, L18, L19, L2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
