File: PCB/half.kicad_sch (KiCad schematic)
At the start: 124 parts, among them J3 JST_PH, SW1 SW_Push, SW10 SW_Push, SW11 SW_Push, SW12 SW_Push, SW13 SW_Push, SW14 SW_Push, SW15 SW_Push, SW16 SW_Push, SW17 SW_Push, SW18 SW_Push, SW19 SW_Push, SW2 SW_Push, SW20 SW_Push, SW21 SW_Push, SW22 SW_Push, SW23 SW_Push, SW24 SW_Push, SW25 SW_Push, SW26 SW_Push, SW27 SW_Push, SW28 SW_Push, SW29 SW_Push, SW3 SW_Push, SW4 SW_Push, SW5 SW_Push, SW6 SW_Push, SW7 SW_Push, SW8 SW_Push, SW9 SW_Push, U3 SuperMini nRF52840

Commit message: routed again
Parts:
- added C59: C_Polarized_Small, Capacitor_Tantalum_SMD:CP_EIA-7343-31_Kemet-D_HandSolder, symbol Device:C_Polarized_Small
- added R1: R_470Ω, Resistor_SMD:R_0805_2012Metric_Pad1.20x1.40mm_HandSolder, symbol Device:R
- C1: value C_Small -> C_Small_0.1uF; footprint (none) -> Capacitor_SMD:C_0805_2012Metric_Pad1.18x1.45mm_HandSolder
- C10, C11, C12, C13, C14, C15, C16, C17, C18, C19, C2, C20, C21, C22, C23, C24, C25, C26, C27, C28, C29, C3, C4, C5, C6, C7, C8, C9: value C_Small -> C_Small_0.1uf; footprint (none) -> Capacitor_SMD:C_0805_2012Metric_Pad1.18x1.45mm_HandSolder
Connections:
- net +3.3V: now also C59.1
- net GND: now also C59.2
- net LED_DAT: now also R1.2; no longer L6.3 (DIN)
- new net: L6.3 (DIN), R1.1
